Commit message: Gazebo related changes.

File: p2os_urdf/defs/pioneer3at.xacro (robot description, xacro)
@@ -8,9 +8,9 @@
 	<link name="base_link">
 		<inertial>
-			<mass value="3.5"/>
-			<origin xyz="-0.025 0 -0.223"/>
-			<inertia ixx="1" ixy="0" ixz="0"
-				 iyy="1" iyz="0"
-				 izz="1"/>
+			<mass value="10.0"/>
+			<origin xyz="0 0 0.177"/>
+			<inertia ixx="0.3338" ixy="0.0" ixz="0.0"
+				 iyy="0.4783" iyz="0.0"
+				 izz="0.3338"/>
 		</inertial>
 		<visual name="base_visual">
@@ -24,7 +24,7 @@
 		</visual>
 		<collision>
-			<origin xyz="0 0 0" rpy="0 0 0"/>
+			<origin xyz="0 0 0.177" rpy="0 0 0"/>
 				<geometry>
-					<box size="0.01 0.01 0.01"/>
+					<mesh filename="package://p2os_urdf/meshes/p3at_meshes/chassis.stl"/>
 				</geometry>
 		</collision>
@@ -33,9 +33,9 @@
 	<link name="top_plate">
 		<inertial>
-			<mass value="0"/>
+			<mass value="0.1"/>
 			<origin xyz="-0.025 0 -0.223"/>
-			<inertia ixx="1" ixy="0" ixz="0"
-				 iyy="1" iyz="0"
- 				izz="1"/>
+			<inertia ixx="1.0" ixy="0.0" ixz="0.0"
+				 iyy="1.0" iyz="0.0"
+ 				izz="1.0"/>
 		</inertial>
 		<visual name="base_visual">
@@ -63,8 +63,8 @@
 	<link name="front_sonar">
 		<inertial>
-			<mass value="0"/>
-			<origin xyz="0 0 0"/>
-			<inertia ixx="1" ixy="0" ixz="0"
-				 iyy="1" iyz="0" izz="1"/>
+			<mass value="0.1"/>
+			<origin xyz="0 0 0"/>
+			<inertia ixx="1.0" ixy="0.0" ixz="0.0"
+				 iyy="1.0" iyz="0.0" izz="1.0"/>
 		</inertial>
 		<visual name="base_visual">
@@ -91,8 +91,8 @@
 	<link name="back_sonar">
 		<inertial>
-			<mass value="0"/>
-			<origin xyz="0 0 0"/>
-			<inertia ixx="1" ixy="0" ixz="0"
-				 iyy="1" iyz="0" izz="1"/>
+			<mass value="0.1"/>
+			<origin xyz="0 0 0"/>
+			<inertia ixx="1.0" ixy="0.0" ixz="0.0"
+				 iyy="1.0" iyz="0.0" izz="1.0"/>
 		</inertial>
 		<visual name="base_visual">
@@ -121,8 +121,8 @@
 	<link name="p3at_front_${suffix}_axle">
 		<inertial>
-			<mass value="0"/>
-			<origin xyz="0 0 0"/>
-			<inertia ixx="1" ixy="0" ixz="0"
-				 iyy="1" iyz="0" izz="1"/>
+			<mass value="0.1"/>
+			<origin xyz="0 0 0"/>
+			<inertia ixx="1.0" ixy="0.0" ixz="0.0"
+				 iyy="1.0" iyz="0.0" izz="1.0"/>
   	 	</inertial>
 	<visual name="base_visual">
@@ -149,8 +149,8 @@
 	<link name="p3at_front_${suffix}_hub">
 		<inertial>
-			<mass value="0"/>
-			<origin xyz="0 0 0"/>
-			<inertia ixx="1" ixy="0" ixz="0"
-				 iyy="1" iyz="0" izz="1"/>
+			<mass value="0.1"/>
+			<origin xyz="0 0 0"/>
+			<inertia ixx="1.0" ixy="0.0" ixz="0.0"
+				 iyy="1.0" iyz="0.0" izz="1.0"/>
   	 	</inertial>
 	<visual name="base_visual">
@@ -177,9 +177,9 @@
 	<link name="p3at_front_${suffix}_wheel">
 		<inertial>
-			<mass value="0"/>
-			<origin xyz="0 0 0"/>
-			<inertia ixx="1" ixy="0" ixz="0"
-				 iyy="1" iyz="0" izz="1"/>
-  	 	</inertial>
+			<mass value="0.5"/>
+			<origin xyz="0 0 0"/>
+			<inertia ixx="0.012411765597" ixy="0" ixz="0"
+         iyy="0.015218160428" iyz="0" izz="0.011763977943"/>
+      </inertial>
 	<visual name="base_visual">
 		<origin xyz="0 0 0" rpy="0 0 0"/>
@@ -194,9 +194,13 @@
 		<origin xyz="0 0 0" rpy="0 0 0"/>
 		<geometry>
-			<box size="0 0 0"/>
-		</geometry>
-	</collision>
-	</link>
-	<joint name="base_front_${suffix}_wheel_joint" type="fixed">
+			<mesh filename="package://p2os_urdf/meshes/p3at_meshes/wheel.stl"/>
+		</geometry>
+	</collision>
+	</link>
+	<joint name="p3at_front_${suffix}_wheel_joint" type="continuous">
+  	<axis xyz="0 1 0"/>
+    <anchor xyz="0 0 0"/>
+    <limit effort="100" velocity="100" />
+    <joint_properties damping="0.7"/>
 		<origin xyz="0 0 0" rpy="0 0 0"/>
 		<parent link="p3at_front_${suffix}_hub"/>
@@ -206,8 +210,8 @@
 	<link name="p3at_back_${suffix}_axle">
 		<inertial>
-			<mass value="0"/>
-			<origin xyz="0 0 0"/>
-			<inertia ixx="1" ixy="0" ixz="0"
-				 iyy="1" iyz="0" izz="1"/>
+			<mass value="0.1"/>
+			<origin xyz="0 0 0"/>
+			<inertia ixx="1.0" ixy="0.0" ixz="0.0"
+				 iyy="1.0" iyz="0.0" izz="1.0"/>
   	 	</inertial>
 	<visual name="base_visual">
@@ -223,5 +227,5 @@
 		<origin xyz="0 0 0" rpy="0 0 0"/>
 		<geometry>
-			<box size="0 0 0"/>
+			<mesh filename="package://p2os_urdf/meshes/p3at_meshes/axle.stl"/>
 		</geometry>
 	</collision>
@@ -234,8 +238,8 @@
 	<link name="p3at_back_${suffix}_hub">
 		<inertial>
-			<mass value="0"/>
-			<origin xyz="0 0 0"/>
-			<inertia ixx="1" ixy="0" ixz="0"
-				 iyy="1" iyz="0" izz="1"/>
+			<mass value="0.1"/>
+			<origin xyz="0 0 0"/>
+			<inertia ixx="1.0" ixy="0.0" ixz="0.0"
+				 iyy="1.0" iyz="0.0" izz="1.0"/>
   	 	</inertial>
 	<visual name="base_visual">
@@ -249,5 +253,5 @@
 		<origin xyz="0 0 0" rpy="0 0 0"/>
 		<geometry>
-			<box size="0 0 0"/>
+			<mesh filename="package://p2os_urdf/meshes/p3at_meshes/${suffix}_hubcap.stl"/>
 		</geometry>
 	</collision>
@@ -260,9 +264,9 @@
 	<link name="p3at_back_${suffix}_wheel">
 		<inertial>
-			<mass value="0"/>
-			<origin xyz="0 0 0"/>
-			<inertia ixx="1" ixy="0" ixz="0"
-				 iyy="1" iyz="0" izz="1"/>
-  	 	</inertial>
+			<mass value="0.5"/>
+			<origin xyz="0 0 0"/>
+			<inertia ixx="0.012411765597" ixy="0" ixz="0"
+         iyy="0.015218160428" iyz="0" izz="0.011763977943"/>
+      </inertial>
 	<visual name="base_visual">
 		<origin xyz="0 0 0" rpy="0 0 0"/>
@@ -275,13 +279,25 @@
 		<origin xyz="0 0 0" rpy="0 0 0"/>
 		<geometry>
-			<box size="0 0 0"/>
-		</geometry>
-	</collision>
-	</link>
-	<joint name="p3at_back_${suffix}_wheel_joint" type="fixed">
+	    <mesh filename="package://p2os_urdf/meshes/p3at_meshes/wheel.stl"/>
+		</geometry>
+	</collision>
+	</link>
+	<joint name="p3at_back_${suffix}_wheel_joint" type="continuous">
+	  <axis xyz="0 1 0"/>
+    <anchor xyz="0 0 0"/>
+    <limit effort="100" velocity="100" />
+    <joint_properties damping="0.7"/>
 		<origin xyz="0 0 0" rpy="0 0 0"/>
 		<parent link="p3at_back_${suffix}_hub"/>
 		<child link="p3at_back_${suffix}_wheel"/>
 	</joint>
+  <gazebo reference="p3at_back_${suffix}_wheel">
+    <mu1>0.2</mu1>
+    <mu2>0.2</mu2>
+  </gazebo>
+  <gazebo reference="p3at_front_${suffix}_wheel">
+    <mu1>0.2</mu1>
+    <mu2>0.2</mu2>
+  </gazebo>
 </xacro:macro>
 <xacro:p3at_front suffix="left" reflect="1"/>
@@ -289,3 +305,20 @@
 <xacro:p3at_back suffix="left" reflect="1"/>
 <xacro:p3at_back suffix="right" reflect="-1"/>
+<gazebo>
+    <plugin name="skid_steer_drive_controller" filename="libgazebo_ros_skid_steer_drive.so">
+        <update>100</update>
+        <updateRate>100.0</updateRate>
+        <robotNamespace>/</robotNamespace>
+        <leftFrontJoint>p3at_front_left_wheel_joint</leftFrontJoint>
+        <rightFrontJoint>p3at_front_right_wheel_joint</rightFrontJoint>
+        <leftRearJoint>p3at_back_left_wheel_joint</leftRearJoint>
+        <rightRearJoint>p3at_back_right_wheel_joint</rightRearJoint>
+        <wheelSeparation>0.4</wheelSeparation>
+        <wheelDiameter>0.215</wheelDiameter>
+        <robotBaseFrame>base_link</robotBaseFrame>
+        <torque>5</torque>
+        <interface:position name="position_iface_0"/>
+        <topicName>cmd_vel</topicName>
+    </plugin>
+</gazebo>
 </robot>

Commit message: URDF of 3AT divided into 2 files.

File: p2os_urdf/defs/pioneer3at.xacro (robot description, xacro)
@@ -5,320 +5,9 @@
        xmlns:xacro="http://ros.org/wiki/xacro"
 name="pioneer3at">
-<!-- Chassis -->
-	<link name="base_link">
-		<inertial>
-			<mass value="10.0"/>
-			<origin xyz="0 0 0.177"/>
-			<inertia ixx="0.3338" ixy="0.0" ixz="0.0"
-				 iyy="0.4783" iyz="0.0"
-				 izz="0.3338"/>
-		</inertial>
-		<visual name="base_visual">
-			<origin xyz="0 0 0.177" rpy="0 0 0"/>
-			<geometry name="pioneer_geom">
-				<mesh filename="package://p2os_urdf/meshes/p3at_meshes/chassis.stl"/>
-			</geometry>
-			<material name="ChassisRed">
-				<color rgba="0.851 0.0 0.0 1.0"/>
-			</material>
-		</visual>
-		<collision>
-			<origin xyz="0 0 0.177" rpy="0 0 0"/>
-				<geometry>
-					<mesh filename="package://p2os_urdf/meshes/p3at_meshes/chassis.stl"/>
-				</geometry>
-		</collision>
-	</link>
-<!-- Top -->
-	<link name="top_plate">
-		<inertial>
-			<mass value="0.1"/>
-			<origin xyz="-0.025 0 -0.223"/>
-			<inertia ixx="1.0" ixy="0.0" ixz="0.0"
-				 iyy="1.0" iyz="0.0"
- 				izz="1.0"/>
-		</inertial>
-		<visual name="base_visual">
-			<origin xyz="0 0 0" rpy="0 0 0"/>
-			<geometry name="pioneer_geom">
-				<mesh filename="package://p2os_urdf/meshes/p3at_meshes/top.stl"/>
-			</geometry>
-			<material name="TopBlack">
-					<color rgba="0.038 0.038 0.038 1.0"/>
-			</material>
-		</visual>
-		<collision>
-			<origin xyz="0 0 0" rpy="0 0 0"/>
-			<geometry>
-				<box size="0 0 0"/>
-			</geometry>
-		</collision>
-	</link>
-	<joint name="base_top_joint" type="fixed">
-		<origin xyz="0.003 0 0.274" rpy="0 0 0"/>
-		<parent link="base_link"/>
-		<child link="top_plate"/>
-	</joint>
-<!-- Front + Back Sonar -->
-	<link name="front_sonar">
-		<inertial>
-			<mass value="0.1"/>
-			<origin xyz="0 0 0"/>
-			<inertia ixx="1.0" ixy="0.0" ixz="0.0"
-				 iyy="1.0" iyz="0.0" izz="1.0"/>
-		</inertial>
-		<visual name="base_visual">
-			<origin xyz="0 0 0" rpy="0 0 0"/>
-			<geometry name="pioneer_geom">
-				<mesh filename="package://p2os_urdf/meshes/p3at_meshes/front_sonar.stl"/>
-			</geometry>
-			<material name="SonarYellow">
-				<color rgba="0.715 0.583 0.210 1.0"/>
-			</material>
-		</visual>
-		<collision>
-			<origin xyz="0 0 0" rpy="0 0 0"/>
-			<geometry>
-				<box size="0 0 0"/>
-			</geometry>
-		</collision>
-	</link>
-	<joint name="base_front_joint" type="fixed">
-		<origin xyz="0.193 0 0.25" rpy="0 0 0"/>
-		<parent link="base_link"/>
-		<child link="front_sonar"/>
-	</joint>
-	<link name="back_sonar">
-		<inertial>
-			<mass value="0.1"/>
-			<origin xyz="0 0 0"/>
-			<inertia ixx="1.0" ixy="0.0" ixz="0.0"
-				 iyy="1.0" iyz="0.0" izz="1.0"/>
-		</inertial>
-		<visual name="base_visual">
-			<origin xyz="0 0 0" rpy="0 0 0"/>
-			<geometry name="pioneer_geom">
-				<mesh filename="package://p2os_urdf/meshes/p3at_meshes/back_sonar.stl"/>
-			</geometry>
-			<material name="SonarYellow">
-				<color rgba="0.715 0.583 0.210 1.0"/>
-			</material>
-		</visual>
-		<collision>
-			<origin xyz="0 0 0" rpy="0 0 0"/>
-			<geometry>
-				<box size="0 0 0"/>
-			</geometry>
-		</collision>
-	</link>
-	<joint name="base_back_joint" type="fixed">
-		<origin xyz="-0.187 0 0.247" rpy="0 0 0"/>
-		<parent link="base_link"/>
-		<child link="back_sonar"/>
-	</joint>
-<!-- Front Axles + Wheels + Hubcaps -->
-<xacro:macro name="p3at_front" params="suffix reflect">
-	<link name="p3at_front_${suffix}_axle">
-		<inertial>
-			<mass value="0.1"/>
-			<origin xyz="0 0 0"/>
-			<inertia ixx="1.0" ixy="0.0" ixz="0.0"
-				 iyy="1.0" iyz="0.0" izz="1.0"/>
-  	 	</inertial>
-	<visual name="base_visual">
-		<origin xyz="0 0 0" rpy="0 0 0"/>
-		<geometry name="pioneer_geom">
-			<mesh filename="package://p2os_urdf/meshes/p3at_meshes/axle.stl"/>
-		</geometry>
-		<material name="AxleGrey">
-			<color rgba="0.5 0.5 0.5 1"/>
-		</material>
-	</visual>
-	<collision>
-		<origin xyz="0 0 0" rpy="0 0 0"/>
-		<geometry>
-			<box size="0 0 0"/>
-		</geometry>
-	</collision>
-	</link>
-	<joint name="base_front_${suffix}_axle_joint" type="fixed">
-		<origin xyz="0.135 ${reflect*0.156} 0.111" rpy="0 0 0"/>
-		<parent link="base_link"/>
-		<child link="p3at_front_${suffix}_axle"/>
-	</joint>
-	<link name="p3at_front_${suffix}_hub">
-		<inertial>
-			<mass value="0.1"/>
-			<origin xyz="0 0 0"/>
-			<inertia ixx="1.0" ixy="0.0" ixz="0.0"
-				 iyy="1.0" iyz="0.0" izz="1.0"/>
-  	 	</inertial>
-	<visual name="base_visual">
-		<origin xyz="0 0 0" rpy="0 0 0"/>
-		<geometry name="pioneer_geom">
-			<mesh filename="package://p2os_urdf/meshes/p3at_meshes/${suffix}_hubcap.stl"/>
-		</geometry>
-		<material name="HubcapYellow">
-			<color rgba="1.0 0.811 0.151 1.0"/>
-		</material>
-	</visual>
-	<collision>
-		<origin xyz="0 0 0" rpy="0 0 0"/>
-		<geometry>
-			<box size="0 0 0"/>
-		</geometry>
-	</collision>
-	</link>
-	<joint name="base_front_${suffix}_hub_joint" type="fixed">
-		<origin xyz="0 ${reflect*0.041} 0" rpy="0 0 0"/>
-		<parent link="p3at_front_${suffix}_axle"/>
-		<child link="p3at_front_${suffix}_hub"/>
-	</joint>
-	<link name="p3at_front_${suffix}_wheel">
-		<inertial>
-			<mass value="0.5"/>
-			<origin xyz="0 0 0"/>
-			<inertia ixx="0.012411765597" ixy="0" ixz="0"
-         iyy="0.015218160428" iyz="0" izz="0.011763977943"/>
-      </inertial>
-	<visual name="base_visual">
-		<origin xyz="0 0 0" rpy="0 0 0"/>
-		<geometry name="pioneer_geom">
-			<mesh filename="package://p2os_urdf/meshes/p3at_meshes/wheel.stl"/>
-		</geometry>
-		<material name="WheelBlack">
-			<color rgba="0.117 0.117 0.117 1"/>
-		</material>
-	</visual>
-	<collision>
-		<origin xyz="0 0 0" rpy="0 0 0"/>
-		<geometry>
-			<mesh filename="package://p2os_urdf/meshes/p3at_meshes/wheel.stl"/>
-		</geometry>
-	</collision>
-	</link>
-	<joint name="p3at_front_${suffix}_wheel_joint" type="continuous">
-  	<axis xyz="0 1 0"/>
-    <anchor xyz="0 0 0"/>
-    <limit effort="100" velocity="100" />
-    <joint_properties damping="0.7"/>
-		<origin xyz="0 0 0" rpy="0 0 0"/>
-		<parent link="p3at_front_${suffix}_hub"/>
-		<child link="p3at_front_${suffix}_wheel"/>
-	</joint>
-<!-- Back Axles + Wheels + Hubcaps -->
-	<link name="p3at_back_${suffix}_axle">
-		<inertial>
-			<mass value="0.1"/>
-			<origin xyz="0 0 0"/>
-			<inertia ixx="1.0" ixy="0.0" ixz="0.0"
-				 iyy="1.0" iyz="0.0" izz="1.0"/>
-  	 	</inertial>
-	<visual name="base_visual">
-		<origin xyz="0 0 0" rpy="0 0 0"/>
-		<geometry name="pioneer_geom">
-			<mesh filename="package://p2os_urdf/meshes/p3at_meshes/axle.stl"/>
-		</geometry>
-		<material name="AxleGrey">
-			<color rgba="0.5 0.5 0.5 1"/>
-		</material>
-	</visual>
-	<collision>
-		<origin xyz="0 0 0" rpy="0 0 0"/>
-		<geometry>
-			<mesh filename="package://p2os_urdf/meshes/p3at_meshes/axle.stl"/>
-		</geometry>
-	</collision>
-	</link>
-	<joint name="bp3at_back_${suffix}_axle_joint" type="fixed">
-		<origin xyz="-0.134 ${reflect*0.156} 0.111" rpy="0 0 0"/>
-		<parent link="base_link"/>
-		<child link="p3at_back_${suffix}_axle"/>
-	</joint>
-	<link name="p3at_back_${suffix}_hub">
-		<inertial>
-			<mass value="0.1"/>
-			<origin xyz="0 0 0"/>
-			<inertia ixx="1.0" ixy="0.0" ixz="0.0"
-				 iyy="1.0" iyz="0.0" izz="1.0"/>
-  	 	</inertial>
-	<visual name="base_visual">
-		<origin xyz="0 0 0" rpy="0 0 0"/>
-		<geometry name="pioneer_geom">
-			<mesh filename="package://p2os_urdf/meshes/p3at_meshes/${suffix}_hubcap.stl"/>
-		</geometry>
-		<material name="HubcapYellow"/>
-	</visual>
-	<collision>
-		<origin xyz="0 0 0" rpy="0 0 0"/>
-		<geometry>
-			<mesh filename="package://p2os_urdf/meshes/p3at_meshes/${suffix}_hubcap.stl"/>
-		</geometry>
-	</collision>
-	</link>
-	<joint name="p3at_back_${suffix}_hub_joint" type="fixed">
-		<origin xyz="-0 ${reflect*0.041} 0" rpy="0 0 0"/>
-		<parent link="p3at_back_${suffix}_axle"/>
-		<child link="p3at_back_${suffix}_hub"/>
-	</joint>
-	<link name="p3at_back_${suffix}_wheel">
-		<inertial>
-			<mass value="0.5"/>
-			<origin xyz="0 0 0"/>
-			<inertia ixx="0.012411765597" ixy="0" ixz="0"
-         iyy="0.015218160428" iyz="0" izz="0.011763977943"/>
-      </inertial>
-	<visual name="base_visual">
-		<origin xyz="0 0 0" rpy="0 0 0"/>
-		<geometry name="pioneer_geom">
-			<mesh filename="package://p2os_urdf/meshes/p3at_meshes/wheel.stl"/>
-		</geometry>
-		<material name="WheelBlack"/>
-	</visual>
-	<collision>
-		<origin xyz="0 0 0" rpy="0 0 0"/>
-		<geometry>
-	    <mesh filename="package://p2os_urdf/meshes/p3at_meshes/wheel.stl"/>
-		</geometry>
-	</collision>
-	</link>
-	<joint name="p3at_back_${suffix}_wheel_joint" type="continuous">
-	  <axis xyz="0 1 0"/>
-    <anchor xyz="0 0 0"/>
-    <limit effort="100" velocity="100" />
-    <joint_properties damping="0.7"/>
-		<origin xyz="0 0 0" rpy="0 0 0"/>
-		<parent link="p3at_back_${suffix}_hub"/>
-		<child link="p3at_back_${suffix}_wheel"/>
-	</joint>
-  <gazebo reference="p3at_back_${suffix}_wheel">
-    <mu1>0.2</mu1>
-    <mu2>0.2</mu2>
-  </gazebo>
-  <gazebo reference="p3at_front_${suffix}_wheel">
-    <mu1>0.2</mu1>
-    <mu2>0.2</mu2>
-  </gazebo>
-</xacro:macro>
+<include filename="$(find p2os_urdf)/defs/pioneer3at_body.xacro"/>
 <xacro:p3at_front suffix="left" reflect="1"/>
 <xacro:p3at_front suffix="right" reflect="-1"/>
 <xacro:p3at_back suffix="left" reflect="1"/>
 <xacro:p3at_back suffix="right" reflect="-1"/>
-<gazebo>
-    <plugin name="skid_steer_drive_controller" filename="libgazebo_ros_skid_steer_drive.so">
-        <update>100</update>
-        <updateRate>100.0</updateRate>
-        <robotNamespace>/</robotNamespace>
-        <leftFrontJoint>p3at_front_left_wheel_joint</leftFrontJoint>
-        <rightFrontJoint>p3at_front_right_wheel_joint</rightFrontJoint>
-        <leftRearJoint>p3at_back_left_wheel_joint</leftRearJoint>
-        <rightRearJoint>p3at_back_right_wheel_joint</rightRearJoint>
-        <wheelSeparation>0.4</wheelSeparation>
-        <wheelDiameter>0.215</wheelDiameter>
-        <robotBaseFrame>base_link</robotBaseFrame>
-        <torque>5</torque>
-        <interface:position name="position_iface_0"/>
-        <topicName>cmd_vel</topicName>
-    </plugin>
-</gazebo>
+<xacro:p3at_gazebo_ext/>
 </robot>
