Commit message: Remove visual names in wheel descriptions...
...due to SDF bug https://bitbucket.org/osrf/sdformat/issues/132/parser-does-not-handle-urdf-material

File: p2os_urdf/defs/pioneer3dx_wheel.xacro (robot description, xacro)
@@ -18,5 +18,5 @@
          iyy="0.015218160428" iyz="0" izz="0.011763977943"/>
       </inertial>
-    <visual name="base_visual">
+    <visual>
       <origin xyz="0 0 0" rpy="0 0 0"/>
       <geometry name="pioneer_geom">
@@ -48,5 +48,5 @@
          iyy="0.015218160428" iyz="0" izz="0.011763977943"/>
       </inertial>
-  <visual name="base_visual">
+  <visual>
     <origin xyz="0 0 0" rpy="0 0 0"/>
     <geometry name="pioneer_geom">

Commit message: Remove deprecated elem tag.
Promote its attributes mu1, mu2, kp, kd to tags.

File: p2os_urdf/defs/pioneer3dx_wheel.xacro (robot description, xacro)
@@ -73,12 +73,12 @@
   </joint>
   <gazebo reference="p3dx_${suffix}_hubcap">
-      <material value="Gazebo/Yellow"/>
+    <material value="Gazebo/Yellow"/>
   </gazebo>
   <gazebo reference="p3dx_${suffix}_wheel">
       <material value="Gazebo/Black"/>
-      <elem key="mu1" value="0.5" />
-      <elem key="mu2" value="50.0" />
-      <elem key="kp"  value="100000000.0" />
-      <elem key="kd"  value="1.0" />
+      <mu1>0.5</mu1>
+      <mu2>50.0</mu2>
+      <kp>100000000.0</kp>
+      <kd>1.0</kd>
   </gazebo>
 </xacro:macro>
