Commit message: Fixed the p2os_urdf.launch to work correctly

File: p2os_urdf/defs/pioneer3dx.xacro (robot description, xacro)
@@ -132,6 +132,6 @@
 		<child link="center_hubcap"/>
 	</joint>
-		<link name="left_hub">
-			<visual>
+	<link name="left_hub">
+		<visual>
 			<origin xyz="0 0 0" rpy="0 0 0"/>
 			<geometry>
@@ -141,14 +141,14 @@
 				<color rgba="1.0 0.811 0.151 1.0"/>
 			</material>
-			</visual>
-		</link>
-		<joint name="left_hub_joint" type="fixed">
-			<origin xyz="0 0.15 0.08" rpy="0 0 0"/>
-			<parent link="base_link"/>
-			<child link="left_hub"/>
-			<axis xyz="0 1 0"/>
-		</joint>
-		<link name="left_wheel_joint">
-			<visual>
+		</visual>
+	</link>
+	<joint name="left_hub_joint" type="fixed">
+		<origin xyz="0 0.15 0.08" rpy="0 0 0"/>
+		<parent link="base_link"/>
+		<child link="left_hub"/>
+		<axis xyz="0 1 0"/>
+	</joint>
+	<link name="left_wheel_joint">
+		<visual>
 			<origin xyz="0 0 0" rpy="0 0 0"/>
 			<geometry>
@@ -158,13 +158,13 @@
 				<color rgba="0.117 0.117 0.117 1"/>
 			</material>
-			</visual>
-		</link>
-		<joint name="left_wheel_joint" type="fixed">
-			<origin xyz="0 0 0" rpy="0 0 0"/>
-			<parent link="left_hub"/>
-			<child link="left_wheel_joint"/>
-		</joint>
-		<link name="right_hub">
-			<visual>
+		</visual>
+	</link>
+	<joint name="left_wheel_joint" type="fixed">
+		<origin xyz="0 0 0" rpy="0 0 0"/>
+		<parent link="left_hub"/>
+		<child link="left_wheel_joint"/>
+	</joint>
+	<link name="right_hub">
+		<visual>
 			<origin xyz="0 0 0" rpy="0 0 0"/>
 			<geometry>
@@ -174,14 +174,14 @@
 				<color rgba="1.0 0.811 0.151 1.0"/>
 			</material>
-			</visual>
-		</link>
-		<joint name="right_hub_joint" type="fixed">
-			<origin xyz="0 -0.15 0.08" rpy="0 0 0"/>
-			<parent link="base_link"/>
-			<child link="right_hub"/>
-			<axis xyz="0 1 0"/>
-		</joint>
-		<link name="right_wheel_joint">
-			<visual>
+		</visual>
+	</link>
+	<joint name="right_hub_joint" type="fixed">
+		<origin xyz="0 -0.15 0.08" rpy="0 0 0"/>
+		<parent link="base_link"/>
+		<child link="right_hub"/>
+		<axis xyz="0 1 0"/>
+	</joint>
+	<link name="right_wheel_joint">
+		<visual>
 			<origin xyz="0 0 0" rpy="0 0 0"/>
 			<geometry>
@@ -191,11 +191,11 @@
 				<color rgba="0.117 0.117 0.117 1"/>
 			</material>
-			</visual>
-		</link>
-		<joint name="right_wheel_joint" type="fixed">
-			<origin xyz="0 0 0" rpy="0 0 0"/>
-			<parent link="right_hub"/>
-			<child link="right_wheel_joint"/>
-		</joint>
+		</visual>
+	</link>
+	<joint name="right_wheel_joint" type="fixed">
+		<origin xyz="0 0 0" rpy="0 0 0"/>
+		<parent link="right_hub"/>
+		<child link="right_wheel_joint"/>
+	</joint>
 <!-- Front + Back Sonar -->
 	<link name="front_sonar">

Commit message: Adding inertia for Gazebo simulation

File: p2os_urdf/defs/pioneer3dx.xacro (robot description, xacro)
@@ -18,4 +18,7 @@
 		</visual>
 	</link>
+	<gazebo reference="base_link">
+		<material value="Gazebo/Red"/>
+	</gazebo>
 <!-- Top -->
 	<joint name="base_top_joint" type="fixed">
@@ -26,4 +29,11 @@
 	<link name="top_plate">
 		<visual>
+			<inertial>
+				<mass value="0.01"/>
+				<origin xyz="0 0 0"/>
+				<inertia ixx="1" ixy="0" ixz="0"
+					 iyy="1" iyz="0"
+	 				izz="1"/>
+			</inertial>
 			<origin xyz="0 0 0" rpy="0 0 0"/>
 			<geometry name="top_geom">
@@ -35,4 +45,7 @@
 		</visual>
 	</link>
+	<gazebo reference="top_plate">
+		<material value="Gazebo/Black"/>
+	</gazebo>
 <!-- Swivel -->
 	<joint name="base_swivel_joint" type="continuous">
@@ -67,4 +80,7 @@
 	</collision>
 	</link>
+	<gazebo reference="swivel">
+		<material value="Gazebo/Grey"/>
+	</gazebo>
 <!-- Center Wheel + Hubcap -->
 	<link name="center_hubcap">

Commit message: Updated the Pioneer-3dx to work with Gazebo in Hydro

File: p2os_urdf/defs/pioneer3dx.xacro (robot description, xacro)
@@ -143,4 +143,7 @@
 	</collision>
 	</link>
+	<gazebo reference="left_hub">
+		<material value="Gazebo/Yellow"/>
+	</gazebo>
 	<joint name="center_wheel_joint" type="fixed">
 		<origin xyz="-0.0035 0 -0.001" rpy="0 0 0"/>
@@ -181,4 +184,7 @@
 		<child link="left_wheel_joint"/>
 	</joint>
+	<gazebo reference="left_wheel_joint">
+		<material value="Gazebo/Black"/>
+	</gazebo>
 	<link name="right_hub">
 		<visual>
@@ -192,4 +198,7 @@
 		</visual>
 	</link>
+	<gazebo reference="right_hub">
+		<material value="Gazebo/Yellow"/>
+	</gazebo>
 	<joint name="right_hub_joint" type="fixed">
 		<origin xyz="0 -0.15 0.08" rpy="0 0 0"/>
@@ -214,4 +223,7 @@
 		<child link="right_wheel_joint"/>
 	</joint>
+	<gazebo reference="right_wheel_joint">
+		<material value="Gazebo/Black"/>
+	</gazebo>
 <!-- Front + Back Sonar -->
 	<link name="front_sonar">
@@ -277,34 +289,18 @@
 		<child link="back_sonar"/>
 	</joint>
-  <gazebo>
-    <controller:diffdrive_plugin name="differential_drive_controller" plugin="libdiffdrive_plugin.so">
-      <alwaysOn>true</alwaysOn>
-      <update>100</update>
-      <updateRate>100.0</updateRate>
-      <leftJoint>base_right_wheel_joint</leftJoint>
-      <rightJoint>base_left_wheel_joint</rightJoint>
-      <wheelSeparation>0.39</wheelSeparation>
-      <wheelDiameter>0.15</wheelDiameter>
-      <torque>5</torque>
-      <interface:position name="position_iface_0"/>
-      <robotNamespace>/</robotNamespace>
-      <topicName>cmd_vel</topicName>
-    </controller:diffdrive_plugin>
-    <controller:gazebo_ros_p3d name="p3d_base_controller" plugin="libgazebo_ros_p3d.so">
-      <alwaysOn>true</alwaysOn>
-      <updateRate>100.0</updateRate>
-      <bodyName>base_link</bodyName>
-      <topicName>base_pose_ground_truth</topicName>
-      <gaussianNoise>0.01</gaussianNoise>
-      <frameName>map</frameName>
-      <xyzOffsets>0 0 0</xyzOffsets> <!-- initialize odometry for fake localization-->
-      <rpyOffsets>0 0 0</rpyOffsets>
-      <interface:position name="p3d_base_position"/>
-    </controller:gazebo_ros_p3d>
-    <controller:gazebo_ros_controller_manager name="gazebo_ros_controller_manager" plugin="libgazebo_ros_controller_manager.so">
-      <alwaysOn>true</alwaysOn>
-      <updateRate>1000.0</updateRate>
-      <interface:audio name="gazebo_ros_controller_manager_dummy_iface" />
-    </controller:gazebo_ros_controller_manager>
-  </gazebo>
+<xacro:macro name="p3at_gazebo_ext">
+<gazebo>
+  <plugin name="skid_steer_drive_controller" filename="libgazebo_ros_skid_steer_drive.so">
+    <updateRate>100.0</updateRate>
+    <robotNamespace>/</robotNamespace>
+    <leftJoint>base_right_wheel_joint</leftJoint>
+    <rightJoint>base_left_wheel_joint</rightJoint>
+    <wheelSeparation>0.39</wheelSeparation>
+    <wheelDiameter>0.15</wheelDiameter>
+    <robotBaseFrame>base_link</robotBaseFrame>
+    <torque>200</torque>
+    <topicName>cmd_vel</topicName>
+  </plugin>
+</gazebo>
+</xacro:macro>
 </robot>

Commit message: Pioneer-3dx circus bug is now fixed. Now to get it to move... We'll see.

File: p2os_urdf/defs/pioneer3dx.xacro (robot description, xacro)
@@ -1,306 +1,11 @@
 <?xml version="1.0"?>
-<robot name="pioneer3dx"
-	xmlns:sensor="http://playerstage.sourceforge.net/gazebo/xmlschema/#sensor"
-	xmlns:controller="http://playerstage.sourceforge.net/gazebo/xmlschema/#controller"
-	xmlns:interface="http://playerstage.sourceforge.net/gazebo/xmlschema/#interface"
-	xmlns:xacro="http://ros.org/wiki/xacro">
-  <include filename="$(find p2os_urdf)/defs/pioneer3dx_wheel.xacro"/>
-<!-- Chassis -->
-	<link name="base_link">
-		<visual name="base_visual">
-			<origin xyz="-0.045 0 0.148" rpy="0 0 0"/>
-			<geometry name="pioneer_geom">
-				<mesh filename="package://p2os_urdf/meshes/p3dx_meshes/chassis.stl"/>
-			</geometry>
-			<material name="ChassisRed">
-				<color rgba="0.851 0.0 0.0 1.0"/>
-			</material>
-		</visual>
-	</link>
-	<gazebo reference="base_link">
-		<material value="Gazebo/Red"/>
-	</gazebo>
-<!-- Top -->
-	<joint name="base_top_joint" type="fixed">
-		<origin xyz="-0.045 0 0.234" rpy="0 0 0"/>
-		<parent link="base_link"/>
-		<child link="top_plate"/>
-	</joint>
-	<link name="top_plate">
-		<visual>
-			<inertial>
-				<mass value="0.01"/>
-				<origin xyz="0 0 0"/>
-				<inertia ixx="1" ixy="0" ixz="0"
-					 iyy="1" iyz="0"
-	 				izz="1"/>
-			</inertial>
-			<origin xyz="0 0 0" rpy="0 0 0"/>
-			<geometry name="top_geom">
-				<mesh filename="package://p2os_urdf/meshes/p3dx_meshes/top.stl"/>
-			</geometry>
-			<material name="TopBlack">
-					<color rgba="0.038 0.038 0.038 1.0"/>
-			</material>
-		</visual>
-	</link>
-	<gazebo reference="top_plate">
-		<material value="Gazebo/Black"/>
-	</gazebo>
-<!-- Swivel -->
-	<joint name="base_swivel_joint" type="continuous">
-		<origin xyz="-0.185 0 0.055" rpy="0 0 0"/>
-		<anchor xyz="0 0 0"/>
-    	<limit effort="100" velocity="100" k_velocity="0" />
-    	<joint_properties damping="0.0" friction="0.0" />
-		<parent link="base_link"/>
-		<child link="swivel"/>
-	</joint>
-	<link name="swivel">
-		<inertial>
-			<mass value="0.1"/>
-			<origin xyz="0 0 0"/>
-			<inertia ixx="0.01" ixy="0" ixz="0"
-				 iyy="0.01" iyz="0" izz="0.01"/>
-  	 	</inertial>
-	<visual name="base_visual">
-		<origin xyz="0 0 0" rpy="0 0 0"/>
-		<geometry name="pioneer_geom">
-			<mesh filename="package://p2os_urdf/meshes/p3dx_meshes/swivel.stl"/>
-		</geometry>
-		<material name="swivel">
-			<color rgba="0.5 0.5 0.5 1"/>
-		</material>
-	</visual>
-	<collision>
-		<origin xyz="0 0 0" rpy="0 0 0"/>
-		<geometry>
-			<box size="0 0 0"/>
-		</geometry>
-	</collision>
-	</link>
-	<gazebo reference="swivel">
-		<material value="Gazebo/Grey"/>
-	</gazebo>
-<!-- Center Wheel + Hubcap -->
-	<link name="center_hubcap">
-		<inertial>
-			<mass value="0.01"/>
-			<origin xyz="0 0 0"/>
-			<inertia ixx="0.012411765597" ixy="-0.000711733678" ixz="0.00050272983"
-				 iyy="0.015218160428" iyz="-0.000004273467" izz="0.011763977943"/>
-  	 	</inertial>
-	<visual name="base_visual">
-		<origin xyz="0 0 0" rpy="0 0 0"/>
-		<geometry name="pioneer_geom">
-			<mesh filename="package://p2os_urdf/meshes/p3dx_meshes/center_hubcap.stl"/>
-		</geometry>
-		<material name="swivel">
-			<color rgba="0.5 0.5 0.5 1"/>
-		</material>
-	</visual>
-	<collision>
-		<origin xyz="0 0 0" rpy="0 0 0"/>
-		<geometry>
-			<box size="0 0 0"/>
-		</geometry>
-	</collision>
-	</link>
-	<gazebo reference="center_hubcap">
-		<material value="Gazebo/Grey"/>
-	</gazebo>
-	<joint name="swivel_hubcap_joint" type="continuous">
-		<origin xyz="-0.026 0 -0.016" rpy="0 0 0"/>
-		<axis xyz="0 1 0"/>
-		<anchor xyz="0 0 0"/>
-    <limit effort="100" velocity="100" k_velocity="0" />
-    <joint_properties damping="0.0" friction="0.0" />
-	  <parent link="swivel"/>
-		<child link="center_wheel"/>
-	</joint>
-	<link name="center_wheel">
-		<inertial>
-			<mass value="0.1"/>
-			<origin xyz="0 0 0"/>
-			<inertia ixx="0.012411765597" ixy="-0.000711733678" ixz="0.00050272983"
-				 iyy="0.015218160428" iyz="-0.000004273467" izz="0.011763977943"/>
-  	 	</inertial>
-	<visual name="base_visual">
-		<origin xyz="0 0 0" rpy="0 0 0"/>
-		<geometry name="pioneer_geom">
-			<mesh filename="package://p2os_urdf/meshes/p3dx_meshes/center_wheel.stl"/>
-		</geometry>
-		<material name="WheelBlack">
-			<color rgba="0.117 0.117 0.117 1"/>
-		</material>
-	</visual>
-	<collision>
-		<origin xyz="0 0 0" rpy="${-3.1415927/2.0} 0 0"/>
-		<geometry>
-			<!--<mesh filename="package://p2os_urdf/meshes/p3dx_meshes/center_wheel.stl"/>-->
-			<cylinder radius="0.0375" length="0.01"/>
-		</geometry>
-	</collision>
-	</link>
-	<gazebo reference="left_hub">
-		<material value="Gazebo/Yellow"/>
-	</gazebo>
-	<joint name="center_wheel_joint" type="fixed">
-		<origin xyz="-0.0035 0 -0.001" rpy="0 0 0"/>
-		<parent link="center_wheel"/>
-		<child link="center_hubcap"/>
-	</joint>
-	<link name="left_hub">
-		<visual>
-			<origin xyz="0 0 0" rpy="0 0 0"/>
-			<geometry>
-				<mesh filename="package://p2os_urdf/meshes/p3dx_meshes/left_hubcap.stl"/>
-			</geometry>
-			<material name="HubcapYellow">
-				<color rgba="1.0 0.811 0.151 1.0"/>
-			</material>
-		</visual>
-	</link>
-	<joint name="left_hub_joint" type="fixed">
-		<origin xyz="0 0.15 0.08" rpy="0 0 0"/>
-		<parent link="base_link"/>
-		<child link="left_hub"/>
-		<axis xyz="0 1 0"/>
-	</joint>
-	<link name="left_wheel_joint">
-		<visual>
-			<origin xyz="0 0 0" rpy="0 0 0"/>
-			<geometry>
-				<mesh filename="package://p2os_urdf/meshes/p3dx_meshes/left_wheel.stl"/>
-			</geometry>
-			<material name="WheelBlack">
-				<color rgba="0.117 0.117 0.117 1"/>
-			</material>
-		</visual>
-	</link>
-	<joint name="left_wheel_joint" type="fixed">
-		<origin xyz="0 0 0" rpy="0 0 0"/>
-		<parent link="left_hub"/>
-		<child link="left_wheel_joint"/>
-	</joint>
-	<gazebo reference="left_wheel_joint">
-		<material value="Gazebo/Black"/>
-	</gazebo>
-	<link name="right_hub">
-		<visual>
-			<origin xyz="0 0 0" rpy="0 0 0"/>
-			<geometry>
-				<mesh filename="package://p2os_urdf/meshes/p3dx_meshes/right_hubcap.stl"/>
-			</geometry>
-			<material name="HubcapYellow">
-				<color rgba="1.0 0.811 0.151 1.0"/>
-			</material>
-		</visual>
-	</link>
-	<gazebo reference="right_hub">
-		<material value="Gazebo/Yellow"/>
-	</gazebo>
-	<joint name="right_hub_joint" type="fixed">
-		<origin xyz="0 -0.15 0.08" rpy="0 0 0"/>
-		<parent link="base_link"/>
-		<child link="right_hub"/>
-		<axis xyz="0 1 0"/>
-	</joint>
-	<link name="right_wheel_joint">
-		<visual>
-			<origin xyz="0 0 0" rpy="0 0 0"/>
-			<geometry>
-				<mesh filename="package://p2os_urdf/meshes/p3dx_meshes/right_wheel.stl"/>
-			</geometry>
-			<material name="WheelBlack">
-				<color rgba="0.117 0.117 0.117 1"/>
-			</material>
-		</visual>
-	</link>
-	<joint name="right_wheel_joint" type="fixed">
-		<origin xyz="0 0 0" rpy="0 0 0"/>
-		<parent link="right_hub"/>
-		<child link="right_wheel_joint"/>
-	</joint>
-	<gazebo reference="right_wheel_joint">
-		<material value="Gazebo/Black"/>
-	</gazebo>
-<!-- Front + Back Sonar -->
-	<link name="front_sonar">
-		<inertial>
-			<mass value="0.0001"/>
-			<origin xyz="0 0 0"/>
-			<inertia ixx="1" ixy="0" ixz="0"
-				 iyy="1" iyz="0" izz="1"/>
-		</inertial>
-		<visual name="base_visual">
-			<origin xyz="0 0 0" rpy="0 0 0"/>
-			<geometry name="pioneer_geom">
-				<mesh filename="package://p2os_urdf/meshes/p3dx_meshes/front_sonar.stl"/>
-			</geometry>
-			<material name="SonarYellow">
-				<color rgba="0.715 0.583 0.210 1.0"/>
-			</material>
-		</visual>
-		<collision>
-			<origin xyz="0 0 0" rpy="0 0 0"/>
-			<geometry>
-				<box size="0 0 0"/>
-			</geometry>
-		</collision>
-	</link>
-	<gazebo reference="front_sonar">
-		<material value="Gazebo/Yellow"/>
-	</gazebo>
-	<joint name="base_front_joint" type="fixed">
-		<origin xyz="-0.198 0 0.208" rpy="0 0 0"/>
-		<parent link="base_link"/>
-		<child link="front_sonar"/>
-	</joint>
-	<link name="back_sonar">
-		<inertial>
-			<mass value="0.0001"/>
-			<origin xyz="0 0 0"/>
-			<inertia ixx="1" ixy="0" ixz="0"
-				 iyy="1" iyz="0" izz="1"/>
-		</inertial>
-		<visual name="back_sonar_vis">
-			<origin xyz="0 0 0" rpy="0 0 0"/>
-			<geometry name="pioneer_geom">
-				<mesh filename="package://p2os_urdf/meshes/p3dx_meshes/back_sonar.stl"/>
-			</geometry>
-			<material name="SonarYellow">
-				<color rgba="0.715 0.583 0.210 1.0"/>
-			</material>
-		</visual>
-		<collision>
-			<origin xyz="0 0 0" rpy="0 0 0"/>
-			<geometry>
-				<box size="0 0 0"/>
-			</geometry>
-		</collision>
-	</link>
-	<gazebo reference="back_sonar">
-		<material value="Gazebo/Yellow"/>
-	</gazebo>
-	<joint name="base_back_joint" type="fixed">
-		<origin xyz="0.109 0 0.209" rpy="0 0 0"/>
-		<parent link="base_link"/>
-		<child link="back_sonar"/>
-	</joint>
-<xacro:macro name="p3at_gazebo_ext">
-<gazebo>
-  <plugin name="skid_steer_drive_controller" filename="libgazebo_ros_skid_steer_drive.so">
-    <updateRate>100.0</updateRate>
-    <robotNamespace>/</robotNamespace>
-    <leftJoint>base_right_wheel_joint</leftJoint>
-    <rightJoint>base_left_wheel_joint</rightJoint>
-    <wheelSeparation>0.39</wheelSeparation>
-    <wheelDiameter>0.15</wheelDiameter>
-    <robotBaseFrame>base_link</robotBaseFrame>
-    <torque>200</torque>
-    <topicName>cmd_vel</topicName>
-  </plugin>
-</gazebo>
-</xacro:macro>
+<robot xmlns:sensor="http://playerstage.sourceforge.net/gazebo/xmlschema/#sensor"
+	   xmlns:controller="http://playerstage.sourceforge.net/gazebo/xmlschema/#controller"
+	   xmlns:interface="http://playerstage.sourceforge.net/gazebo/xmlschema/#interface"
+	   xmlns:xacro="http://ros.org/wiki/xacro"
+	   name="pioneer3dx">
+	<include filename="$(find p2os_urdf)/defs/pioneer3dx_body.xacro"/>
+	<!-- <xacro:right_wheel_joint suffix="" reflect="1"/>
+	<xacro:left_wheel_joint suffix="" reflect="-1"/>
+	<xacro:p3dx_gazebo_ext/> -->
 </robot>

Commit message: Fix xacro deprecated warnings.

File: p2os_urdf/defs/pioneer3dx.xacro (robot description, xacro)
@@ -5,5 +5,5 @@
 	   xmlns:xacro="http://ros.org/wiki/xacro"
 	   name="pioneer3dx">
-	<include filename="$(find p2os_urdf)/defs/pioneer3dx_body.xacro"/>
+	<xacro:include filename="$(find p2os_urdf)/defs/pioneer3dx_body.xacro"/>
 	<!-- <xacro:right_wheel_joint suffix="" reflect="1"/>
 	<xacro:left_wheel_joint suffix="" reflect="-1"/>

File: p2os_urdf/defs/pioneer3dx_body.xacro (robot description, xacro)
@@ -1,10 +1,9 @@
 <?xml version="1.0"?>
 <robot xmlns:sensor="http://playerstage.sourceforge.net/gazebo/xmlschema/#sensor"
-	   xmlns:controller="http://playerstage.sourceforge.net/gazebo/
-	   xmlschema/#controller"
+	   xmlns:controller="http://playerstage.sourceforge.net/gazebo/xmlschema/#controller"
 	   xmlns:interface="http://playerstage.sourceforge.net/gazebo/xmlschema/#interface"
 	   xmlns:xacro="http://ros.org/wiki/xacro"
 	   >
-	<include filename="$(find p2os_urdf)/defs/pioneer3dx_wheel.xacro"/>
+	<xacro:include filename="$(find p2os_urdf)/defs/pioneer3dx_wheel.xacro"/>
 	<!-- Chassis description -->
 	<link name="base_link">

File: p2os_urdf/defs/pioneer3dx_wheel.xacro (robot description, xacro)
@@ -6,7 +6,7 @@
   xmlns:xacro="http://ros.org/wiki/xacro"
   >
-  <!--<include filename="$(find p2os_urdf)/defs/materials.xacro"/>-->
+  <!--<xacro:include filename="$(find p2os_urdf)/defs/materials.xacro"/>-->
   <!-- Properties (Constants) -->
-  <property name="M_PI" value="3.14159"/>
+  <xacro:property name="M_PI" value="3.14159"/>
 <!-- Right/Left Hubcap + Wheel -->
 <xacro:macro name="p3dx_wheel" params="suffix parent reflect">

Commit message: Clean up obsolete xml-schema namespaces.

File: p2os_urdf/defs/pioneer3dx.xacro (robot description, xacro)
@@ -1,11 +1,4 @@
 <?xml version="1.0"?>
-<robot xmlns:sensor="http://playerstage.sourceforge.net/gazebo/xmlschema/#sensor"
-	   xmlns:controller="http://playerstage.sourceforge.net/gazebo/xmlschema/#controller"
-	   xmlns:interface="http://playerstage.sourceforge.net/gazebo/xmlschema/#interface"
-	   xmlns:xacro="http://ros.org/wiki/xacro"
-	   name="pioneer3dx">
+<robot name="pioneer3dx" xmlns:xacro="http://ros.org/wiki/xacro">
 	<xacro:include filename="$(find p2os_urdf)/defs/pioneer3dx_body.xacro"/>
-	<!-- <xacro:right_wheel_joint suffix="" reflect="1"/>
-	<xacro:left_wheel_joint suffix="" reflect="-1"/>
-	<xacro:p3dx_gazebo_ext/> -->
 </robot>

File: p2os_urdf/defs/pioneer3dx_body.xacro (robot description, xacro)
@@ -1,8 +1,4 @@
 <?xml version="1.0"?>
-<robot xmlns:sensor="http://playerstage.sourceforge.net/gazebo/xmlschema/#sensor"
-	   xmlns:controller="http://playerstage.sourceforge.net/gazebo/xmlschema/#controller"
-	   xmlns:interface="http://playerstage.sourceforge.net/gazebo/xmlschema/#interface"
-	   xmlns:xacro="http://ros.org/wiki/xacro"
-	   >
+<robot xmlns:xacro="http://ros.org/wiki/xacro">
 	<xacro:include filename="$(find p2os_urdf)/defs/pioneer3dx_wheel.xacro"/>
 	<!-- Chassis description -->

File: p2os_urdf/defs/pioneer3dx_wheel.xacro (robot description, xacro)
@@ -1,9 +1,4 @@
 <?xml version="1.0"?>
-<robot
-  xmlns:sensor="http://playerstage.sourceforge.net/gazebo/xmlschema/#sensor"
-  xmlns:controller="http://playerstage.sourceforge.net/gazebo/xmlschema/#controller"
-  xmlns:interface="http://playerstage.sourceforge.net/gazebo/xmlschema/#interface"
-  xmlns:xacro="http://ros.org/wiki/xacro"
-  >
+<robot xmlns:xacro="http://ros.org/wiki/xacro">
   <!--<xacro:include filename="$(find p2os_urdf)/defs/materials.xacro"/>-->
   <!-- Properties (Constants) -->
@@ -30,5 +25,4 @@
       <origin xyz="0 0 0" rpy="${-3.1415927/2} 0 0"/>
       <geometry>
-        <!--<mesh filename="package://p2os_urdf/meshes/p3dx_meshes/${suffix}_wheel.stl"/>-->
         <cylinder radius="0.09" length="0.04"/>
       </geometry>
@@ -36,5 +30,4 @@
   </link>
   <joint name="base_${suffix}_hubcap_joint" type="fixed">
-    <!--<origin xyz="0 ${reflect*0.158} 0.091" rpy="0 0 0"/>-->
     <origin xyz="0 0 0" rpy="0 0 0"/>
     <parent link="p3dx_${suffix}_wheel"/>
@@ -58,4 +51,5 @@
   </visual>
   </link>
+  <!-- The transmission tag is used only by ros_control -->
   <!--<transmission type="pr2_mechanism_model/SimpleTransmission" name="${parent}_${suffix}_wheel_trans">
     <actuator name="base_${suffix}_wheel_motor" />
