Commit message: Clean up indentation.

File: p2os_urdf/defs/pioneer3dx.xacro (robot description, xacro)
@@ -1,4 +1,4 @@
 <?xml version="1.0"?>
 <robot name="pioneer3dx" xmlns:xacro="http://ros.org/wiki/xacro">
-	<xacro:include filename="$(find p2os_urdf)/defs/pioneer3dx_body.xacro"/>
+  <xacro:include filename="$(find p2os_urdf)/defs/pioneer3dx_body.xacro"/>
 </robot>

File: p2os_urdf/defs/pioneer3dx_body.xacro (robot description, xacro)
@@ -1,243 +1,243 @@
 <?xml version="1.0"?>
 <robot xmlns:xacro="http://ros.org/wiki/xacro">
-	<xacro:include filename="$(find p2os_urdf)/defs/pioneer3dx_wheel.xacro"/>
-	<!-- Chassis description -->
-	<link name="base_link">
-		<!-- CHECK THESE VALUES. THEY MAY BE COMPLETELY WRONG. -->
-		<inertial>
-			<mass value="40.0"/>
-			<origin xyz="-0.045 0 0.148"/>
-			<inertia ixx="0.3338" ixy="0.0" ixz="0.0"
-				 iyy="0.4783" iyz="0.0"
-				 izz="0.3338"/>
-		</inertial>
-		<!-- The base visual is fine. Just the inertial is questionable.-->
-		<visual>
-			<origin xyz="-0.045 0 0.148" rpy="0 0 0"/>
-			<geometry name="pioneer_geom">
-				<mesh filename="package://p2os_urdf/meshes/p3dx_meshes/chassis.stl"/>
-			</geometry>
-			<material name="ChassisRed">
-				<color rgba="0.851 0.0 0.0 1.0"/>
-			</material>
-		</visual>
-		<collision>
-			<origin xyz="-0.045 0 0.148" rpy="0 0 0"/>
-			<geometry>
-              <box size="0.4 0.28 0.17"/>
-              <!-- This is the correct bounding box, but x=0.43 crashes Gazebo? -->
-			  <!--box size="0.43 0.28 0.17"/-->
-			</geometry>
-		</collision>
-	</link>
-	<gazebo reference="base_link">
-		<material value="Gazebo/Red"/>
-	</gazebo>
-	<link name="top_plate">
-		<inertial>
-			<mass value="0.01"/>
-			<origin xyz="0 0 0"/>
-			<inertia ixx="1" ixy="0" ixz="0"
-				 iyy="1" iyz="0"
- 				izz="1"/>
-		</inertial>
-		<visual>
-			<origin xyz="0 0 0" rpy="0 0 0"/>
-			<geometry name="pioneer_geom">
-				<mesh filename="package://p2os_urdf/meshes/p3dx_meshes/top.stl"/>
-			</geometry>
-			<material name="TopBlack">
-					<color rgba="0.038 0.038 0.038 1.0"/>
-			</material>
-		</visual>
-	</link>
-	<gazebo reference="top_plate">
-		<material value="Gazebo/Black"/>
-	</gazebo>
-	<joint name="base_top_joint" type="fixed">
-		<origin xyz="-0.045 0 0.24" rpy="0 0 0"/>
-		<parent link="base_link"/>
-		<child link="top_plate"/>
-	</joint>
-	<!-- Swivel -->
-	<link name="swivel">
-		<inertial>
-			<mass value="0.1"/>
-			<origin xyz="0 0 0"/>
-			<inertia ixx="0.01" ixy="0" ixz="0"
-				 iyy="0.01" iyz="0" izz="0.01"/>
-  	 	</inertial>
-	<visual>
-		<origin xyz="0 0 0" rpy="0 0 0"/>
-		<geometry name="pioneer_geom">
-			<mesh filename="package://p2os_urdf/meshes/p3dx_meshes/swivel.stl"/>
-		</geometry>
-		<material name="swivel">
-			<color rgba="0.5 0.5 0.5 1"/>
-		</material>
-	</visual>
-	</link>
-	<gazebo reference="swivel">
-		<material value="Gazebo/Black"/>
-	</gazebo>
-    <joint name="base_swivel_joint" type="continuous">
-		<origin xyz="-0.185 0 0.055" rpy="0 0 0"/>
-		<axis xyz="0 0 1"/>
-    	<limit effort="100" velocity="100" k_velocity="0" />
-    	<joint_properties damping="0.0" friction="0.0" />
-		<parent link="base_link"/>
-		<child link="swivel"/>
-	</joint>
-<!-- Center Wheel + Hubcap -->
-	<link name="center_hubcap">
-		<inertial>
-			<mass value="0.01"/>
-			<origin xyz="0 0 0"/>
-			<inertia ixx="0.012411765597" ixy="-0.000711733678" ixz="0.00050272983"
-				 iyy="0.015218160428" iyz="-0.000004273467" izz="0.011763977943"/>
-  	 	</inertial>
-	<visual>
-		<origin xyz="0 0 0" rpy="0 0 0"/>
-		<geometry name="pioneer_geom">
-			<mesh filename="package://p2os_urdf/meshes/p3dx_meshes/center_hubcap.stl"/>
-		</geometry>
-		<material name="swivel">
-			<color rgba="0.5 0.5 0.5 1"/>
-		</material>
-	</visual>
-	</link>
-	<gazebo reference="center_hubcap">
-		<material value="Gazebo/Black"/>
-	</gazebo>
-	<joint name="swivel_hubcap_joint" type="continuous">
-		<origin xyz="-0.026 0 -0.016" rpy="0 0 0"/>
-		<axis xyz="0 1 0"/>
-		<anchor xyz="0 0 0"/>
+  <xacro:include filename="$(find p2os_urdf)/defs/pioneer3dx_wheel.xacro"/>
+  <!-- Chassis description -->
+  <link name="base_link">
+	<!-- CHECK THESE VALUES. THEY MAY BE COMPLETELY WRONG. -->
+	<inertial>
+	  <mass value="40.0"/>
+	  <origin xyz="-0.045 0 0.148"/>
+	  <inertia ixx="0.3338" ixy="0.0" ixz="0.0"
+			   iyy="0.4783" iyz="0.0"
+			   izz="0.3338"/>
+	</inertial>
+	<!-- The base visual is fine. Just the inertial is questionable.-->
+	<visual>
+	  <origin xyz="-0.045 0 0.148" rpy="0 0 0"/>
+	  <geometry name="pioneer_geom">
+		<mesh filename="package://p2os_urdf/meshes/p3dx_meshes/chassis.stl"/>
+	  </geometry>
+	  <material name="ChassisRed">
+		<color rgba="0.851 0.0 0.0 1.0"/>
+	  </material>
+	</visual>
+	<collision>
+	  <origin xyz="-0.045 0 0.148" rpy="0 0 0"/>
+	  <geometry>
+        <box size="0.4 0.28 0.17"/>
+        <!-- This is the correct bounding box, but x=0.43 crashes Gazebo? -->
+		<!--box size="0.43 0.28 0.17"/-->
+	  </geometry>
+	</collision>
+  </link>
+  <gazebo reference="base_link">
+	<material value="Gazebo/Red"/>
+  </gazebo>
+  <link name="top_plate">
+	<inertial>
+	  <mass value="0.01"/>
+	  <origin xyz="0 0 0"/>
+	  <inertia ixx="1" ixy="0" ixz="0"
+			   iyy="1" iyz="0"
+ 			   izz="1"/>
+	</inertial>
+	<visual>
+	  <origin xyz="0 0 0" rpy="0 0 0"/>
+	  <geometry name="pioneer_geom">
+		<mesh filename="package://p2os_urdf/meshes/p3dx_meshes/top.stl"/>
+	  </geometry>
+	  <material name="TopBlack">
+		<color rgba="0.038 0.038 0.038 1.0"/>
+	  </material>
+	</visual>
+  </link>
+  <gazebo reference="top_plate">
+	<material value="Gazebo/Black"/>
+  </gazebo>
+  <joint name="base_top_joint" type="fixed">
+	<origin xyz="-0.045 0 0.24" rpy="0 0 0"/>
+	<parent link="base_link"/>
+	<child link="top_plate"/>
+  </joint>
+  <!-- Swivel -->
+  <link name="swivel">
+	<inertial>
+	  <mass value="0.1"/>
+	  <origin xyz="0 0 0"/>
+	  <inertia ixx="0.01" ixy="0" ixz="0"
+			   iyy="0.01" iyz="0" izz="0.01"/>
+  	</inertial>
+	<visual>
+	  <origin xyz="0 0 0" rpy="0 0 0"/>
+	  <geometry name="pioneer_geom">
+		<mesh filename="package://p2os_urdf/meshes/p3dx_meshes/swivel.stl"/>
+	  </geometry>
+	  <material name="swivel">
+		<color rgba="0.5 0.5 0.5 1"/>
+	  </material>
+	</visual>
+  </link>
+  <gazebo reference="swivel">
+	<material value="Gazebo/Black"/>
+  </gazebo>
+  <joint name="base_swivel_joint" type="continuous">
+	<origin xyz="-0.185 0 0.055" rpy="0 0 0"/>
+	<axis xyz="0 0 1"/>
     <limit effort="100" velocity="100" k_velocity="0" />
     <joint_properties damping="0.0" friction="0.0" />
-	  <parent link="swivel"/>
-		<child link="center_wheel"/>
-	</joint>
-	<link name="center_wheel">
-		<inertial>
-			<mass value="0.1"/>
-			<origin xyz="0 0 0"/>
-			<inertia ixx="0.012411765597" ixy="-0.000711733678" ixz="0.00050272983"
-				 iyy="0.015218160428" iyz="-0.000004273467" izz="0.011763977943"/>
-  	 	</inertial>
-	<visual>
-		<origin xyz="0 0 0" rpy="0 0 0"/>
-		<geometry name="pioneer_geom">
-			<mesh filename="package://p2os_urdf/meshes/p3dx_meshes/center_wheel.stl"/>
-		</geometry>
-		<material name="WheelBlack">
-			<color rgba="0.117 0.117 0.117 1"/>
-		</material>
+	<parent link="base_link"/>
+	<child link="swivel"/>
+  </joint>
+  <!-- Center Wheel + Hubcap -->
+  <link name="center_hubcap">
+    <inertial>
+	  <mass value="0.01"/>
+	  <origin xyz="0 0 0"/>
+	  <inertia ixx="0.012411765597" ixy="-0.000711733678" ixz="0.00050272983"
+			   iyy="0.015218160428" iyz="-0.000004273467" izz="0.011763977943"/>
+  	</inertial>
+	<visual>
+	  <origin xyz="0 0 0" rpy="0 0 0"/>
+	  <geometry name="pioneer_geom">
+		<mesh filename="package://p2os_urdf/meshes/p3dx_meshes/center_hubcap.stl"/>
+	  </geometry>
+	  <material name="swivel">
+		<color rgba="0.5 0.5 0.5 1"/>
+	  </material>
+	</visual>
+  </link>
+  <gazebo reference="center_hubcap">
+	<material value="Gazebo/Black"/>
+  </gazebo>
+  <joint name="swivel_hubcap_joint" type="continuous">
+	<origin xyz="-0.026 0 -0.016" rpy="0 0 0"/>
+	<axis xyz="0 1 0"/>
+	<anchor xyz="0 0 0"/>
+    <limit effort="100" velocity="100" k_velocity="0" />
+    <joint_properties damping="0.0" friction="0.0" />
+	<parent link="swivel"/>
+	<child link="center_wheel"/>
+  </joint>
+  <link name="center_wheel">
+	<inertial>
+	  <mass value="0.1"/>
+	  <origin xyz="0 0 0"/>
+	  <inertia ixx="0.012411765597" ixy="-0.000711733678" ixz="0.00050272983"
+			   iyy="0.015218160428" iyz="-0.000004273467" izz="0.011763977943"/>
+  	</inertial>
+	<visual>
+	  <origin xyz="0 0 0" rpy="0 0 0"/>
+	  <geometry name="pioneer_geom">
+		<mesh filename="package://p2os_urdf/meshes/p3dx_meshes/center_wheel.stl"/>
+	  </geometry>
+	  <material name="WheelBlack">
+		<color rgba="0.117 0.117 0.117 1"/>
+	  </material>
 	</visual>
 	<collision>
-		<origin xyz="0 0 0" rpy="${-3.1415927/2.0} 0 0"/>
-		<geometry>
-			<!--<mesh filename="package://p2os_urdf/meshes/p3dx_meshes/center_wheel.stl"/>-->
-			<cylinder radius="0.0375" length="0.0314"/>
-		</geometry>
+	  <origin xyz="0 0 0" rpy="${-3.1415927/2.0} 0 0"/>
+	  <geometry>
+		<!--<mesh filename="package://p2os_urdf/meshes/p3dx_meshes/center_wheel.stl"/>-->
+		<cylinder radius="0.0375" length="0.0314"/>
+	  </geometry>
 	</collision>
-	</link>
-	<gazebo reference="center_wheel">
-		<material value="Gazebo/Black"/>
-	</gazebo>
-	<joint name="center_wheel_joint" type="fixed">
-		<origin xyz="-0.0035 0 -0.001" rpy="0 0 0"/>
-		<parent link="center_wheel"/>
-		<child link="center_hubcap"/>
-	</joint>
-    <xacro:p3dx_wheel suffix="left" parent="base_link" reflect="1"/>
-    <xacro:p3dx_wheel suffix="right" parent="base_link" reflect="-1"/>
-	<!-- Front + Back Sonar -->
-	<link name="front_sonar">
-		<inertial>
-			<mass value="0.0001"/>
-			<origin xyz="0 0 0"/>
-			<inertia ixx="1" ixy="0" ixz="0"
-				 iyy="1" iyz="0" izz="1"/>
-		</inertial>
-		<visual>
-			<origin xyz="0 0 0" rpy="0 0 0"/>
-			<geometry name="pioneer_geom">
-				<mesh filename="package://p2os_urdf/meshes/p3dx_meshes/front_sonar.stl"/>
-			</geometry>
-			<material name="SonarYellow">
-				<color rgba="0.715 0.583 0.210 1.0"/>
-			</material>
-		</visual>
-	</link>
-	<gazebo reference="front_sonar">
-		<material value="Gazebo/Yellow"/>
-	</gazebo>
-	<joint name="base_front_joint" type="fixed">
-		<origin xyz="-0.198 0 0.208" rpy="0 0 0"/>
-		<parent link="base_link"/>
-		<child link="front_sonar"/>
-	</joint>
-	<link name="back_sonar">
-		<inertial>
-			<mass value="0.0001"/>
-			<origin xyz="0 0 0"/>
-			<inertia ixx="1" ixy="0" ixz="0"
-				 iyy="1" iyz="0" izz="1"/>
-		</inertial>
-		<visual>
-			<origin xyz="0 0 0" rpy="0 0 0"/>
-			<geometry name="pioneer_geom">
-				<mesh filename="package://p2os_urdf/meshes/p3dx_meshes/back_sonar.stl"/>
-			</geometry>
-			<material name="SonarYellow">
-				<color rgba="0.715 0.583 0.210 1.0"/>
-			</material>
-		</visual>
-	</link>
-	<gazebo reference="back_sonar">
-		<material value="Gazebo/Yellow"/>
-	</gazebo>
-	<joint name="base_back_joint" type="fixed">
-		<origin xyz="0.109 0 0.209" rpy="0 0 0"/>
-		<!-- <origin xyz="0 0 0" rpy="0 0 0"/> -->
-		<parent link="base_link"/>
-		<child link="back_sonar"/>
-	</joint>
-	<gazebo>
-      <!-- Robot locomotion plugin -->
-	  <plugin name="differential_drive_controller" filename="libgazebo_ros_diff_drive.so">
-        <legacyMode>false</legacyMode>
-        <alwaysOn>true</alwaysOn>
-	    <updateRate>100.0</updateRate>
-	    <leftJoint>base_left_wheel_joint</leftJoint>
-        <rightJoint>base_right_wheel_joint</rightJoint>
-	    <wheelSeparation>0.32</wheelSeparation>
-	    <wheelDiameter>0.18</wheelDiameter>
-	    <wheelTorque>5</wheelTorque>
-        <wheelAcceleration>0</wheelAcceleration>
-        <robotNamespace>pioneer</robotNamespace>
-	    <commandTopic>cmd_vel</commandTopic>
-	    <odometryTopic>odom</odometryTopic>
-        <odometrySource>ENCODER</odometrySource><!--Other option is World-->
-	    <odometryFrame>odom</odometryFrame>
-        <robotBaseFrame>base_link</robotBaseFrame>
-        <publishTf>1</publishTf>
-        <publishWheelTF>false</publishWheelTF>
-        <publishWheelJointState>false</publishWheelJointState>
-        <rosDebugLevel>Warn</rosDebugLevel>
-	  </plugin>
-      <!-- Fake localization plugin -->
-      <plugin name="ground_truth_odometry" filename="libgazebo_ros_p3d.so">
-		<alwaysOn>true</alwaysOn>
-		<updateRate>100.0</updateRate>
-		<bodyName>base_link</bodyName>
-		<topicName>base_pose_ground_truth</topicName>
-		<gaussianNoise>0.01</gaussianNoise>
-		<frameName>map</frameName>-->
-        <!-- initialize odometry for fake localization-->
-		<xyzOffsets>0 0 0</xyzOffsets>
-		<rpyOffsets>0 0 0</rpyOffsets>
-	  </plugin>
-	</gazebo>
+  </link>
+  <gazebo reference="center_wheel">
+	<material value="Gazebo/Black"/>
+  </gazebo>
+  <joint name="center_wheel_joint" type="fixed">
+	<origin xyz="-0.0035 0 -0.001" rpy="0 0 0"/>
+	<parent link="center_wheel"/>
+	<child link="center_hubcap"/>
+  </joint>
+  <xacro:p3dx_wheel suffix="left" parent="base_link" reflect="1"/>
+  <xacro:p3dx_wheel suffix="right" parent="base_link" reflect="-1"/>
+  <!-- Front + Back Sonar -->
+  <link name="front_sonar">
+	<inertial>
+	  <mass value="0.0001"/>
+	  <origin xyz="0 0 0"/>
+	  <inertia ixx="1" ixy="0" ixz="0"
+			   iyy="1" iyz="0" izz="1"/>
+	</inertial>
+	<visual>
+	  <origin xyz="0 0 0" rpy="0 0 0"/>
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
File: p2os_urdf/defs/pioneer3dx_wheel.xacro (robot description, xacro)
@@ -4,70 +4,70 @@
   <!-- Properties (Constants) -->
   <xacro:property name="M_PI" value="3.14159"/>
-<!-- Right/Left Hubcap + Wheel -->
-<xacro:macro name="p3dx_wheel" params="suffix parent reflect">
-  <link name="p3dx_${suffix}_wheel">
-    <inertial>
-      <mass value="0.5"/>
-      <origin xyz="0 0 0"/>
-      <inertia ixx="0.012411765597" ixy="0" ixz="0"
-         iyy="0.015218160428" iyz="0" izz="0.011763977943"/>
+  <!-- Right/Left Hubcap + Wheel -->
+  <xacro:macro name="p3dx_wheel" params="suffix parent reflect">
+    <link name="p3dx_${suffix}_wheel">
+      <inertial>
+        <mass value="0.5"/>
+        <origin xyz="0 0 0"/>
+        <inertia ixx="0.012411765597" ixy="0" ixz="0"
+                 iyy="0.015218160428" iyz="0" izz="0.011763977943"/>
       </inertial>
-    <visual>
+      <visual>
+        <origin xyz="0 0 0" rpy="0 0 0"/>
+        <geometry name="pioneer_geom">
+          <mesh filename="package://p2os_urdf/meshes/p3dx_meshes/${suffix}_wheel.stl"/>
+        </geometry>
+        <material name="WheelBlack">
+          <color rgba="0.117 0.117 0.117 1"/>
+        </material>
+      </visual>
+      <collision>
+        <origin xyz="0 0 0" rpy="${-3.1415927/2} 0 0"/>
+        <geometry>
+          <cylinder radius="0.09" length="0.04"/>
+        </geometry>
+      </collision>
+    </link>
+    <joint name="base_${suffix}_hubcap_joint" type="fixed">
       <origin xyz="0 0 0" rpy="0 0 0"/>
-      <geometry name="pioneer_geom">
-        <mesh filename="package://p2os_urdf/meshes/p3dx_meshes/${suffix}_wheel.stl"/>
-      </geometry>
-      <material name="WheelBlack">
-        <color rgba="0.117 0.117 0.117 1"/>
-      </material>
-    </visual>
-    <collision>
-      <origin xyz="0 0 0" rpy="${-3.1415927/2} 0 0"/>
-      <geometry>
-        <cylinder radius="0.09" length="0.04"/>
-      </geometry>
-    </collision>
-  </link>
-  <joint name="base_${suffix}_hubcap_joint" type="fixed">
-    <origin xyz="0 0 0" rpy="0 0 0"/>
-    <parent link="p3dx_${suffix}_wheel"/>
-    <child link="p3dx_${suffix}_hubcap"/>
-  </joint>
-  <link name="p3dx_${suffix}_hubcap">
-    <inertial>
-      <mass value="0.01"/>
-      <origin xyz="0 0 0"/>
-      <inertia ixx="0.012411765597" ixy="0" ixz="0"
-         iyy="0.015218160428" iyz="0" izz="0.011763977943"/>
+      <parent link="p3dx_${suffix}_wheel"/>
+      <child link="p3dx_${suffix}_hubcap"/>
+    </joint>
+    <link name="p3dx_${suffix}_hubcap">
+      <inertial>
+        <mass value="0.01"/>
+        <origin xyz="0 0 0"/>
+        <inertia ixx="0.012411765597" ixy="0" ixz="0"
+                 iyy="0.015218160428" iyz="0" izz="0.011763977943"/>
       </inertial>
-  <visual>
-    <origin xyz="0 0 0" rpy="0 0 0"/>
-    <geometry name="pioneer_geom">
-      <mesh filename="package://p2os_urdf/meshes/p3dx_meshes/${suffix}_hubcap.stl"/>
-    </geometry>
-    <material name="HubcapYellow">
-      <color rgba="1.0 0.811 0.151 1.0"/>
-    </material>
-  </visual>
-  </link>
-  <!-- The transmission tag is used only by ros_control -->
-  <!--<transmission type="pr2_mechanism_model/SimpleTransmission" name="${parent}_${suffix}_wheel_trans">
-    <actuator name="base_${suffix}_wheel_motor" />
-    <joint name="base_${suffix}_wheel_joint" />
-    <mechanicalReduction>${reflect * 624/35 * 80/19}</mechanicalReduction>
-  </transmission>-->
-  <joint name="base_${suffix}_wheel_joint" type="continuous">
-    <axis xyz="0 1 0"/>
-    <anchor xyz="0 0 0"/>
-    <limit effort="100" velocity="100" />
-    <joint_properties damping="0.0" friction="0.0" />
-    <origin xyz="0 ${reflect*0.158} 0.091" rpy="0 0 0"/>
-    <parent link="base_link"/>
-    <child link="p3dx_${suffix}_wheel"/>
-  </joint>
-  <gazebo reference="p3dx_${suffix}_hubcap">
-    <material value="Gazebo/Yellow"/>
-  </gazebo>
-  <gazebo reference="p3dx_${suffix}_wheel">
+      <visual>
+        <origin xyz="0 0 0" rpy="0 0 0"/>
+        <geometry name="pioneer_geom">
+          <mesh filename="package://p2os_urdf/meshes/p3dx_meshes/${suffix}_hubcap.stl"/>
+        </geometry>
+        <material name="HubcapYellow">
+          <color rgba="1.0 0.811 0.151 1.0"/>
+        </material>
+      </visual>
+    </link>
+    <!-- The transmission tag is used only by ros_control -->
+    <!--<transmission type="pr2_mechanism_model/SimpleTransmission" name="${parent}_${suffix}_wheel_trans">
+        <actuator name="base_${suffix}_wheel_motor" />
+        <joint name="base_${suffix}_wheel_joint" />
+        <mechanicalReduction>${reflect * 624/35 * 80/19}</mechanicalReduction>
+        </transmission>-->
+    <joint name="base_${suffix}_wheel_joint" type="continuous">
+      <axis xyz="0 1 0"/>
+      <anchor xyz="0 0 0"/>
+      <limit effort="100" velocity="100" />
+      <joint_properties damping="0.0" friction="0.0" />
+      <origin xyz="0 ${reflect*0.158} 0.091" rpy="0 0 0"/>
+      <parent link="base_link"/>
+      <child link="p3dx_${suffix}_wheel"/>
+    </joint>
+    <gazebo reference="p3dx_${suffix}_hubcap">
+      <material value="Gazebo/Yellow"/>
+    </gazebo>
+    <gazebo reference="p3dx_${suffix}_wheel">
       <material value="Gazebo/Black"/>
       <mu1>0.5</mu1>
@@ -75,5 +75,5 @@
       <kp>100000000.0</kp>
       <kd>1.0</kd>
-  </gazebo>
-</xacro:macro>
+    </gazebo>
+  </xacro:macro>
 </robot>
