Commit message: Fix crash on model spawn in Gazebo.
Remove zero-sized collision elements, as per this thread: http://answers.gazebosim.org/question/15816/gazebo-crashes-when-spawning-robot-from-urdf/

File: p2os_urdf/defs/pioneer3dx_body.xacro (robot description, xacro)
@@ -88,10 +88,4 @@
 		</material>
 	</visual>
-	<collision>
-		<origin xyz="0 0 0" rpy="0 0 0"/>
-		<geometry>
-			<box size="0 0 0"/>
-		</geometry>
-	</collision>
 	</link>
 	<gazebo reference="swivel">
@@ -272,10 +266,4 @@
 			</material>
 		</visual>
-		<collision>
-			<origin xyz="0 0 0" rpy="0 0 0"/>
-			<geometry>
-				<box size="0 0 0"/>
-			</geometry>
-		</collision>
 	</link>
 	<gazebo reference="front_sonar">

Commit message: Remove visual names.
Visual names prevented Gazebo from rendering material colors, as per this issue: https://bitbucket.org/osrf/sdformat/issues/132/parser-does-not-handle-urdf-material

File: p2os_urdf/defs/pioneer3dx_body.xacro (robot description, xacro)
@@ -18,5 +18,5 @@
 		</inertial>
 		<!-- The base visual is fine. Just the inertial is questionable.-->
-		<visual name="pioneer_geom">
+		<visual>
 			<origin xyz="-0.045 0 0.148" rpy="0 0 0"/>
 			<geometry name="pioneer_geom">
@@ -45,5 +45,5 @@
  				izz="1"/>
 		</inertial>
-		<visual name="pioneer_geom">
+		<visual>
 			<origin xyz="0 0 0" rpy="0 0 0"/>
 			<geometry name="pioneer_geom">
@@ -79,5 +79,5 @@
 				 iyy="0.01" iyz="0" izz="0.01"/>
   	 	</inertial>
-	<visual name="pioneer_geom">
+	<visual>
 		<origin xyz="0 0 0" rpy="0 0 0"/>
 		<geometry name="pioneer_geom">
@@ -100,5 +100,5 @@
 				 iyy="0.015218160428" iyz="-0.000004273467" izz="0.011763977943"/>
   	 	</inertial>
-	<visual name="pioneer_geom">
+	<visual>
 		<origin xyz="0 0 0" rpy="0 0 0"/>
 		<geometry name="pioneer_geom">
@@ -135,5 +135,5 @@
 				 iyy="0.015218160428" iyz="-0.000004273467" izz="0.011763977943"/>
   	 	</inertial>
-	<visual name="pioneer_geom">
+	<visual>
 		<origin xyz="0 0 0" rpy="0 0 0"/>
 		<geometry name="pioneer_geom">
@@ -257,5 +257,5 @@
 				 iyy="1" iyz="0" izz="1"/>
 		</inertial>
-		<visual name="pioneer_geom">
+		<visual>
 			<origin xyz="0 0 0" rpy="0 0 0"/>
 			<geometry name="pioneer_geom">
@@ -282,5 +282,5 @@
 				 iyy="1" iyz="0" izz="1"/>
 		</inertial>
-		<visual name="back_sonar_vis">
+		<visual>
 			<origin xyz="0 0 0" rpy="0 0 0"/>
 			<geometry name="pioneer_geom">

Commit message: Use wheel descriptions from pioneer3dx_wheel.xacro.
Remove invalid collision element from wheel definition.
Comment out transmission element for now.

File: p2os_urdf/defs/pioneer3dx_body.xacro (robot description, xacro)
@@ -160,93 +160,6 @@
 		<child link="center_hubcap"/>
 	</joint>
-	<link name="left_hub">
-		<visual>
-			<origin xyz="0 0 0" rpy="0 0 0"/>
-			<geometry>
-				<mesh filename="package://p2os_urdf/meshes/p3dx_meshes/left_hubcap.stl"/>
-			</geometry>
-			<material name="HubcapYellow">
-				<color rgba="1.0 0.811 0.151 1.0"/>
-			</material>
-		</visual>
-		<collision>
-			<origin xyz="0 0 0" rpy="${-3.1415927/2.0} 0 0"/>
-			<geometry>
-				<!--<mesh filename="package://p2os_urdf/meshes/p3dx_meshes/center_wheel.stl"/>-->
-				<cylinder radius="0.09" length="0.01"/>
-			</geometry>
-		</collision>
-	</link>
-	<joint name="left_hub_joint" type="fixed">
-		<origin xyz="0 0.15 0.08" rpy="0 0 0"/>
-		<parent link="base_link"/>
-		<child link="left_hub"/>
-		<axis xyz="0 1 0"/>
-	</joint>
-	<link name="left_wheel_joint">
-		<visual>
-			<origin xyz="0 0 0" rpy="0 0 0"/>
-			<geometry>
-				<mesh filename="package://p2os_urdf/meshes/p3dx_meshes/left_wheel.stl"/>
-			</geometry>
-			<material name="WheelBlack">
-				<color rgba="0.117 0.117 0.117 1"/>
-			</material>
-		</visual>
-	</link>
-	<joint name="left_wheel_joint" type="fixed">
-		<origin xyz="0 0 0" rpy="0 0 0"/>
-		<parent link="left_hub"/>
-		<child link="left_wheel_joint"/>
-	</joint>
-	<gazebo reference="left_wheel_joint">
-		<material value="Gazebo/Black"/>
-	</gazebo>
-	<link name="right_hub">
-		<visual>
-			<origin xyz="0 0 0" rpy="0 0 0"/>
-			<geometry>
-				<mesh filename="package://p2os_urdf/meshes/p3dx_meshes/right_hubcap.stl"/>
-			</geometry>
-			<material name="HubcapYellow">
-				<color rgba="1.0 0.811 0.151 1.0"/>
-			</material>
-		</visual>
-		<collision>
-		<origin xyz="0 0 0" rpy="${-3.1415927/2.0} 0 0"/>
-		<geometry>
-			<!--<mesh filename="package://p2os_urdf/meshes/p3dx_meshes/center_wheel.stl"/>-->
-			<cylinder radius="0.09" length="0.01"/>
-		</geometry>
-	</collision>
-	</link>
-	<gazebo reference="right_hub">
-		<material value="Gazebo/Yellow"/>
-	</gazebo>
-	<joint name="right_hub_joint" type="fixed">
-		<origin xyz="0 -0.15 0.08" rpy="0 0 0"/>
-		<parent link="base_link"/>
-		<child link="right_hub"/>
-		<axis xyz="0 1 0"/>
-	</joint>
-	<link name="right_wheel_joint">
-		<visual>
-			<origin xyz="0 0 0" rpy="0 0 0"/>
-			<geometry>
-				<mesh filename="package://p2os_urdf/meshes/p3dx_meshes/right_wheel.stl"/>
-			</geometry>
-			<material name="WheelBlack">
-				<color rgba="0.117 0.117 0.117 1"/>
-			</material>
-		</visual>
-	</link>
-	<joint name="right_wheel_joint" type="fixed">
-		<origin xyz="0 0 0" rpy="0 0 0"/>
-		<parent link="right_hub"/>
-		<child link="right_wheel_joint"/>
-	</joint>
-	<gazebo reference="right_wheel_joint">
-		<material value="Gazebo/Black"/>
-	</gazebo>
+    <xacro:p3dx_wheel suffix="left" parent="base_link" reflect="1"/>
+    <xacro:p3dx_wheel suffix="right" parent="base_link" reflect="-1"/>
 	<!-- Front + Back Sonar -->
 	<link name="front_sonar">

File: p2os_urdf/defs/pioneer3dx_wheel.xacro (robot description, xacro)
@@ -57,16 +57,10 @@
     </material>
   </visual>
-  <collision>
-    <origin xyz="0 0 0" rpy="0 0 0"/>
-    <geometry>
-      <box size="0 0 0"/>
-    </geometry>
-  </collision>
   </link>
-  <transmission type="pr2_mechanism_model/SimpleTransmission" name="${parent}_${suffix}_wheel_trans">
+  <!--<transmission type="pr2_mechanism_model/SimpleTransmission" name="${parent}_${suffix}_wheel_trans">
     <actuator name="base_${suffix}_wheel_motor" />
     <joint name="base_${suffix}_wheel_joint" />
     <mechanicalReduction>${reflect * 624/35 * 80/19}</mechanicalReduction>
-  </transmission>
+  </transmission>-->
   <joint name="base_${suffix}_wheel_joint" type="continuous">
     <axis xyz="0 1 0"/>

Commit message: Clean up and simplify collisions.

File: p2os_urdf/defs/pioneer3dx_body.xacro (robot description, xacro)
@@ -28,7 +28,9 @@
 		<collision>
 			<origin xyz="-0.045 0 0.148" rpy="0 0 0"/>
-				<geometry>
-					<mesh filename="package://p2os_urdf/meshes/p3at_meshes/chassis.stl"/>
-				</geometry>
+			<geometry>
+              <box size="0.4 0.28 0.17"/>
+              <!-- This is the correct bounding box, but x=0.43 crashes Gazebo? -->
+			  <!--box size="0.43 0.28 0.17"/-->
+			</geometry>
 		</collision>
 	</link>
@@ -108,10 +110,4 @@
 		</material>
 	</visual>
-	<collision>
-		<origin xyz="0 0 0" rpy="0 0 0"/>
-		<geometry>
-			<box size="0.05 0.05 0.05"/>
-		</geometry>
-	</collision>
 	</link>
 	<gazebo reference="center_hubcap">
@@ -147,5 +143,5 @@
 		<geometry>
 			<!--<mesh filename="package://p2os_urdf/meshes/p3dx_meshes/center_wheel.stl"/>-->
-			<cylinder radius="0.0375" length="0.01"/>
+			<cylinder radius="0.0375" length="0.0314"/>
 		</geometry>
 	</collision>
@@ -203,10 +199,4 @@
 			</material>
 		</visual>
-		<collision>
-			<origin xyz="0 0 0" rpy="0 0 0"/>
-			<geometry>
-				<box size=" 0.5 0.25 0.05"/>
-			</geometry>
-		</collision>
 	</link>
 	<gazebo reference="back_sonar">

File: p2os_urdf/defs/pioneer3dx_wheel.xacro (robot description, xacro)
@@ -31,5 +31,5 @@
       <geometry>
         <!--<mesh filename="package://p2os_urdf/meshes/p3dx_meshes/${suffix}_wheel.stl"/>-->
-        <cylinder radius="0.09" length="0.01"/>
+        <cylinder radius="0.09" length="0.04"/>
       </geometry>
     </collision>

Commit message: Add and configure differential drive plugin.
Seems to behave reasonably.
There is an issue with the swivel which seems to break off randomly.

File: p2os_urdf/defs/pioneer3dx_body.xacro (robot description, xacro)
@@ -209,22 +209,40 @@
 		<child link="back_sonar"/>
 	</joint>
-	<xacro:macro name="p3dx_gazebo_ext">
 	<gazebo>
-	  <plugin name="skid_steer_drive_controller" filename="libgazebo_ros_skid_steer_drive.so">
+      <!-- Robot locomotion plugin -->
+	  <plugin name="differential_drive_controller" filename="libgazebo_ros_diff_drive.so">
+        <legacyMode>false</legacyMode>
+        <alwaysOn>true</alwaysOn>
 	    <updateRate>100.0</updateRate>
-	    <robotNamespace>/</robotNamespace>
-	    <leftFrontJoint>base_swivel_joint</leftFrontJoint>
-	    <rightFrontJoint>base_swivel_joint</rightFrontJoint>
-	    <leftRearJoint>swivel_hubcap_joint</leftRearJoint>
-	    <rightRearJoint>swivel_hubcap_joint</rightRearJoint>
-	    <wheelSeparation>0.3</wheelSeparation>
-	    <wheelDiameter>0.1</wheelDiameter>
-	    <robotBaseFrame>base_link</robotBaseFrame>
-	    <torque>200</torque>
+	    <leftJoint>base_left_wheel_joint</leftJoint>
+        <rightJoint>base_right_wheel_joint</rightJoint>
+	    <wheelSeparation>0.32</wheelSeparation>
+	    <wheelDiameter>0.18</wheelDiameter>
+	    <wheelTorque>5</wheelTorque>
+        <wheelAcceleration>0</wheelAcceleration>
+        <robotNamespace>pioneer</robotNamespace>
 	    <commandTopic>cmd_vel</commandTopic>
 	    <odometryTopic>odom</odometryTopic>
+        <odometrySource>ENCODER</odometrySource><!--Other option is World-->
 	    <odometryFrame>odom</odometryFrame>
+        <robotBaseFrame>base_link</robotBaseFrame>
+        <publishTf>1</publishTf>
+        <publishWheelTF>false</publishWheelTF>
+        <publishWheelJointState>false</publishWheelJointState>
+        <rosDebugLevel>Warn</rosDebugLevel>
 	  </plugin>
-	</gazebo>
-	</xacro:macro>
+      <!-- Fake localization plugin -->
+<!--      <plugin name="p3d_base_controller" plugin="libgazebo_ros_p3d.so">
+		<alwaysOn>true</alwaysOn>
+		<updateRate>100.0</updateRate>
+		<bodyName>base_link</bodyName>
+		<topicName>base_pose_ground_truth</topicName>
+		<gaussianNoise>0.01</gaussianNoise>
+		<frameName>map</frameName>-->
+        <!-- initialize odometry for fake localization-->
+<!--		<xyzOffsets>0 0 0</xyzOffsets>
+		<rpyOffsets>0 0 0</rpyOffsets>
+	  </plugin>
+-->
+	</gazebo>
 </robot>

Commit message: Fix swivel joint.

File: p2os_urdf/defs/pioneer3dx_body.xacro (robot description, xacro)
@@ -65,12 +65,4 @@
 	</joint>
 	<!-- Swivel -->
-	<joint name="base_swivel_joint" type="continuous">
-		<origin xyz="-0.185 0 0.055" rpy="0 0 0"/>
-		<anchor xyz="0 0 0"/>
-    	<limit effort="100" velocity="100" k_velocity="0" />
-    	<joint_properties damping="0.0" friction="0.0" />
-		<parent link="base_link"/>
-		<child link="swivel"/>
-	</joint>
 	<link name="swivel">
 		<inertial>
@@ -91,6 +83,14 @@
 	</link>
 	<gazebo reference="swivel">
-		<material value="Gazebo/Grey"/>
-	</gazebo>
+		<material value="Gazebo/Black"/>
+	</gazebo>
+    <joint name="base_swivel_joint" type="continuous">
+		<origin xyz="-0.185 0 0.055" rpy="0 0 0"/>
+		<axis xyz="0 0 1"/>
+    	<limit effort="100" velocity="100" k_velocity="0" />
+    	<joint_properties damping="0.0" friction="0.0" />
+		<parent link="base_link"/>
+		<child link="swivel"/>
+	</joint>
 <!-- Center Wheel + Hubcap -->
 	<link name="center_hubcap">
@@ -112,5 +112,5 @@
 	</link>
 	<gazebo reference="center_hubcap">
-		<material value="Gazebo/Grey"/>
+		<material value="Gazebo/Black"/>
 	</gazebo>
 	<joint name="swivel_hubcap_joint" type="continuous">
@@ -147,6 +147,6 @@
 	</collision>
 	</link>
-	<gazebo reference="left_hub">
-		<material value="Gazebo/Yellow"/>
+	<gazebo reference="center_wheel">
+		<material value="Gazebo/Black"/>
 	</gazebo>
 	<joint name="center_wheel_joint" type="fixed">

Commit message: Change mass to more reasonable value.

File: p2os_urdf/defs/pioneer3dx_body.xacro (robot description, xacro)
@@ -6,5 +6,5 @@
 	<!-- CHECK THESE VALUES. THEY MAY BE COMPLETELY WRONG. -->
 	<inertial>
-	  <mass value="40.0"/>
+	  <mass value="20.0"/>
 	  <origin xyz="-0.045 0 0.148"/>
 	  <inertia ixx="0.3338" ixy="0.0" ixz="0.0"
