Commit message: Updated the Pioneer-3AT xacro to have colour in Gazebo, and added a launch file.

File: p2os_urdf/defs/pioneer3at_body.xacro (robot description, xacro)
@@ -30,4 +30,7 @@
 		</collision>
 	</link>
+	<gazebo reference="base_link">
+		<material value="Gazebo/Red"/>
+	</gazebo>
 <!-- Top -->
 	<link name="top_plate">
@@ -55,4 +58,7 @@
 		</collision>
 	</link>
+	<gazebo reference="top_plate">
+		<material value="Gazebo/Black"/>
+	</gazebo>
 	<joint name="base_top_joint" type="fixed">
 		<origin xyz="0.003 0 0.274" rpy="0 0 0"/>
@@ -84,4 +90,7 @@
 		</collision>
 	</link>
+	<gazebo reference="front_sonar">
+		<material value="Gazebo/Yellow"/>
+	</gazebo>
 	<joint name="base_front_joint" type="fixed">
 		<origin xyz="0.193 0 0.25" rpy="0 0 0"/>
@@ -112,4 +121,7 @@
 		</collision>
 	</link>
+	<gazebo reference="back_sonar">
+		<material value="Gazebo/Yellow"/>
+	</gazebo>
 	<joint name="base_back_joint" type="fixed">
 		<origin xyz="-0.187 0 0.247" rpy="0 0 0"/>
@@ -142,4 +154,7 @@
 	</collision>
 	</link>
+	<gazebo reference="p3at_front_${suffix}_axle">
+		<material value="Gazebo/Grey"/>
+	</gazebo>
 	<joint name="base_front_${suffix}_axle_joint" type="fixed">
 		<origin xyz="0.135 ${reflect*0.156} 0.111" rpy="0 0 0"/>
@@ -170,4 +185,7 @@
 	</collision>
 	</link>
+	<gazebo reference="p3at_front_${suffix}_hub">
+		<material value="Gazebo/Yellow"/>
+	</gazebo>
 	<joint name="base_front_${suffix}_hub_joint" type="fixed">
 		<origin xyz="0 ${reflect*0.041} 0" rpy="0 0 0"/>
@@ -198,4 +216,7 @@
 	</collision>
 	</link>
+	<gazebo reference="p3at_front_${suffix}_wheel">
+		<material value="Gazebo/Black"/>
+	</gazebo>
 	<joint name="p3at_front_${suffix}_wheel_joint" type="continuous">
   	<axis xyz="0 1 0"/>
@@ -231,4 +252,7 @@
 	</collision>
 	</link>
+	<gazebo reference="p3at_back_${suffix}_axle">
+		<material value="Gazebo/Grey"/>
+	</gazebo>
 	<joint name="bp3at_back_${suffix}_axle_joint" type="fixed">
 		<origin xyz="-0.134 ${reflect*0.156} 0.111" rpy="0 0 0"/>
@@ -257,4 +281,7 @@
 	</collision>
 	</link>
+	<gazebo reference="p3at_back_${suffix}_hub">
+		<material value="Gazebo/Yellow"/>
+	</gazebo>
 	<joint name="p3at_back_${suffix}_hub_joint" type="fixed">
 		<origin xyz="-0 ${reflect*0.041} 0" rpy="0 0 0"/>
@@ -283,4 +310,7 @@
 	</collision>
 	</link>
+	<gazebo reference="p3at_back_${suffix}_wheel">
+		<material value="Gazebo/Black"/>
+	</gazebo>
 	<joint name="p3at_back_${suffix}_wheel_joint" type="continuous">
 	  <axis xyz="0 1 0"/>

Commit message: Changes to wheel collision geometry (robot was unable to rotate).

File: p2os_urdf/defs/pioneer3at_body.xacro (robot description, xacro)
@@ -210,7 +210,9 @@
 	</visual>
 	<collision>
-		<origin xyz="0 0 0" rpy="0 0 0"/>
-		<geometry>
-			<mesh filename="package://p2os_urdf/meshes/p3at_meshes/wheel.stl"/>
+		<origin xyz="0 0 0" rpy="${-3.1415927/2} 0 0"/>
+		<geometry>
+	    <!--mesh filename="package://p2os_urdf/meshes/p3at_meshes/wheel.stl"/-->
+	    <!--cylinder radius="0.111" length="0.075"/-->
+	    <cylinder radius="0.111" length="0.005"/> <!-- workaround -->
 		</geometry>
 	</collision>
@@ -304,7 +306,9 @@
 	</visual>
 	<collision>
-		<origin xyz="0 0 0" rpy="0 0 0"/>
-		<geometry>
-	    <mesh filename="package://p2os_urdf/meshes/p3at_meshes/wheel.stl"/>
+		<origin xyz="0 0 0" rpy="${-3.1415927/2} 0 0"/>
+		<geometry>
+	    <!--mesh filename="package://p2os_urdf/meshes/p3at_meshes/wheel.stl"/-->
+	    <!--cylinder radius="0.111" length="0.075"/-->
+	    <cylinder radius="0.111" length="0.005"/> <!-- workaround -->
 		</geometry>
 	</collision>
@@ -323,10 +327,10 @@
 	</joint>
   <gazebo reference="p3at_back_${suffix}_wheel">
-    <mu1>0.2</mu1>
-    <mu2>0.2</mu2>
+    <mu1>1</mu1>
+    <mu2>1</mu2>
   </gazebo>
   <gazebo reference="p3at_front_${suffix}_wheel">
-    <mu1>0.2</mu1>
-    <mu2>0.2</mu2>
+    <mu1>1</mu1>
+    <mu2>1</mu2>
   </gazebo>
 </xacro:macro>
@@ -344,5 +348,5 @@
     <wheelDiameter>0.215</wheelDiameter>
     <robotBaseFrame>base_link</robotBaseFrame>
-    <torque>5</torque>
+    <torque>200</torque>
     <interface:position name="position_iface_0"/>
     <topicName>cmd_vel</topicName>

Commit message: Changes to wheel collision geometry and Gazebo settings.

File: p2os_urdf/defs/pioneer3at_body.xacro (robot description, xacro)
@@ -213,6 +213,5 @@
 		<geometry>
 	    <!--mesh filename="package://p2os_urdf/meshes/p3at_meshes/wheel.stl"/-->
-	    <!--cylinder radius="0.111" length="0.075"/-->
-	    <cylinder radius="0.111" length="0.005"/> <!-- workaround -->
+	    <cylinder radius="0.111" length="0.075"/>
 		</geometry>
 	</collision>
@@ -309,6 +308,5 @@
 		<geometry>
 	    <!--mesh filename="package://p2os_urdf/meshes/p3at_meshes/wheel.stl"/-->
-	    <!--cylinder radius="0.111" length="0.075"/-->
-	    <cylinder radius="0.111" length="0.005"/> <!-- workaround -->
+	    <cylinder radius="0.111" length="0.075"/>
 		</geometry>
 	</collision>
@@ -327,10 +325,20 @@
 	</joint>
   <gazebo reference="p3at_back_${suffix}_wheel">
-    <mu1>1</mu1>
-    <mu2>1</mu2>
+    <kp>1000000.0</kp> <!-- kp and kd for rubber -->
+    <kd>100.0</kd>
+    <mu1>10.0</mu1>
+    <mu2>1.0</mu2>
+    <fdir1>0 1 0</fdir1> <!-- is this correct? -->
+    <maxVel>1.0</maxVel>
+    <minDepth>0.00</minDepth>
   </gazebo>
   <gazebo reference="p3at_front_${suffix}_wheel">
-    <mu1>1</mu1>
-    <mu2>1</mu2>
+    <kp>1000000.0</kp> <!-- kp and kd for rubber -->
+    <kd>100.0</kd>
+    <mu1>10.0</mu1>
+    <mu2>1.0</mu2>
+    <fdir1>0 1 0</fdir1> <!-- is this correct? -->
+    <maxVel>1.0</maxVel>
+    <minDepth>0.00</minDepth>
   </gazebo>
 </xacro:macro>
@@ -338,5 +346,4 @@
 <gazebo>
   <plugin name="skid_steer_drive_controller" filename="libgazebo_ros_skid_steer_drive.so">
-    <update>100</update>
     <updateRate>100.0</updateRate>
     <robotNamespace>/</robotNamespace>
@@ -349,5 +356,4 @@
     <robotBaseFrame>base_link</robotBaseFrame>
     <torque>200</torque>
-    <interface:position name="position_iface_0"/>
     <topicName>cmd_vel</topicName>
   </plugin>

Commit message: Updated the pioneer3at URDF xacro file. Fixes #38

File: p2os_urdf/defs/pioneer3at_body.xacro (robot description, xacro)
@@ -229,5 +229,7 @@
 		<child link="p3at_front_${suffix}_wheel"/>
 	</joint>
+</xacro:macro>
 <!-- Back Axles + Wheels + Hubcaps -->
+<xacro:macro name="p3at_back" params="suffix reflect">
 	<link name="p3at_back_${suffix}_axle">
 		<inertial>

File: p2os_urdf/defs/pioneer3dx.urdf.xacro (robot description, xacro)
@@ -87,5 +87,5 @@
 	</collision>
 	</link>
- 	<joint name="base_swivel_joint" type="continuous">
+ 	<joint name="base_swivel_joint" type="fixed">
 		<origin xyz="-0.185 0 0.055" rpy="0 0 0"/>
 		<axis xyz="0 0 1" />
@@ -219,4 +219,5 @@
 	<back_sonar parent="base_link"/>
   	<top_plate  parent="base_link"/>
+  	<swivel     parent="base_link"/>
   	</create>
 <gazebo>

Commit message: Fixed color in gazebo with 3at.

File: p2os_urdf/defs/pioneer3at_body.xacro (robot description, xacro)
@@ -14,5 +14,5 @@
 				 izz="0.3338"/>
 		</inertial>
-		<visual name="base_visual">
+		<visual>
 			<origin xyz="0 0 0.177" rpy="0 0 0"/>
 			<geometry name="pioneer_geom">
@@ -42,5 +42,5 @@
  				izz="1.0"/>
 		</inertial>
-		<visual name="base_visual">
+		<visual>
 			<origin xyz="0 0 0" rpy="0 0 0"/>
 			<geometry name="pioneer_geom">
@@ -74,5 +74,5 @@
 				 iyy="1.0" iyz="0.0" izz="1.0"/>
 		</inertial>
-		<visual name="base_visual">
+		<visual>
 			<origin xyz="0 0 0" rpy="0 0 0"/>
 			<geometry name="pioneer_geom">
@@ -105,5 +105,5 @@
 				 iyy="1.0" iyz="0.0" izz="1.0"/>
 		</inertial>
-		<visual name="base_visual">
+		<visual>
 			<origin xyz="0 0 0" rpy="0 0 0"/>
 			<geometry name="pioneer_geom">
@@ -138,5 +138,5 @@
 				 iyy="1.0" iyz="0.0" izz="1.0"/>
   	 	</inertial>
-	<visual name="base_visual">
+	<visual>
 		<origin xyz="0 0 0" rpy="0 0 0"/>
 		<geometry name="pioneer_geom">
@@ -169,5 +169,5 @@
 				 iyy="1.0" iyz="0.0" izz="1.0"/>
   	 	</inertial>
-	<visual name="base_visual">
+	<visual>
 		<origin xyz="0 0 0" rpy="0 0 0"/>
 		<geometry name="pioneer_geom">
@@ -200,5 +200,5 @@
          iyy="0.015218160428" iyz="0" izz="0.011763977943"/>
       </inertial>
-	<visual name="base_visual">
+	<visual>
 		<origin xyz="0 0 0" rpy="0 0 0"/>
 		<geometry name="pioneer_geom">
@@ -239,5 +239,5 @@
 				 iyy="1.0" iyz="0.0" izz="1.0"/>
   	 	</inertial>
-	<visual name="base_visual">
+	<visual>
 		<origin xyz="0 0 0" rpy="0 0 0"/>
 		<geometry name="pioneer_geom">
@@ -270,5 +270,5 @@
 				 iyy="1.0" iyz="0.0" izz="1.0"/>
   	 	</inertial>
-	<visual name="base_visual">
+	<visual>
 		<origin xyz="0 0 0" rpy="0 0 0"/>
 		<geometry name="pioneer_geom">
@@ -299,5 +299,5 @@
          iyy="0.015218160428" iyz="0" izz="0.011763977943"/>
       </inertial>
-	<visual name="base_visual">
+	<visual>
 		<origin xyz="0 0 0" rpy="0 0 0"/>
 		<geometry name="pioneer_geom">
